Commit message: Add manipulator .sdf

File: morus_description/urdf/morus.base.urdf.xacro (robot description, xacro)
@@ -28,4 +28,7 @@
   <xacro:property name="cos45" value="0.7071" />
   <xacro:property name="PI" value="3.14" />
+  <!-- Manipulator properties-->
+  <xacro:property name="link_length" value="0.5" />
+  <xacro:property name="link_mass" value="1" />
   <!-- Property Blocks -->
   <xacro:property name="body_inertia">
@@ -55,4 +58,11 @@
     izz="${(imu_mass * imu_size * imu_size)/6}"
     ixy="0.0" ixz="0.0"  iyz="0.0" /> <!-- [kg*m^2] [kg*m^2] [kg*m^2] [kg*m^2] [kg*m^2] [kg*m^2] -->
+  </xacro:property>
+  <xacro:property name="link_inertia">
+    <inertia
+    ixx="${(link_length * link_mass)/12}"
+    iyy="${(link_length * link_mass)/12}"
+    izz="${(link_length * link_mass)/12}"
+    ixy="0.0" ixz="0.0" iyz="0.0" />
   </xacro:property>
   <!-- Included URDF Files -->
@@ -95,3 +105,83 @@
       <xacro:insert_block name="land_gear_inertia"/>
   </xacro:landing_gear>
+    <!-- Instantiate rotors -->
+  <xacro:vertical_rotor
+    robot_namespace="$(arg name)"
+    suffix="front"
+    direction="cw"
+    motor_constant="${motor_constant}"
+    moment_constant="${moment_constant}"
+    parent="base_link"
+    mass_rotor="${mass_rotor}"
+    radius_rotor="${radius_rotor}"
+    time_constant="${time_constant}"
+    max_rot_velocity="${max_rot_velocity}"
+    motor_number="0"
+    rotor_drag_coefficient="${rotor_drag_coefficient}"
+    rolling_moment_coefficient="${rolling_moment_coefficient}"
+    color="Red">
+    <origin xyz="${arm_length+arm_offset} 0 ${propeler_offset}" rpy="0 0 0" />
+    <xacro:insert_block name="rotor_inertia" />
+  </xacro:vertical_rotor>
+  <xacro:vertical_rotor
+    robot_namespace="$(arg name)"
+    suffix="left"
+    direction="ccw"
+    motor_constant="${motor_constant}"
+    moment_constant="${moment_constant}"
+    parent="base_link"
+    mass_rotor="${mass_rotor}"
+    radius_rotor="${radius_rotor}"
+    time_constant="${time_constant}"
+    max_rot_velocity="${max_rot_velocity}"
+    motor_number="1"
+    rotor_drag_coefficient="${rotor_drag_coefficient}"
+    rolling_moment_coefficient="${rolling_moment_coefficient}"
+    color="Blue">
+    <origin xyz="0 ${arm_length+arm_offset} ${propeler_offset}" rpy="0 0 0" />
+    <xacro:insert_block name="rotor_inertia" />
+  </xacro:vertical_rotor>
+  <xacro:vertical_rotor
+    robot_namespace="$(arg name)"
+    suffix="back"
+    direction="cw"
+    motor_constant="${motor_constant}"
+    moment_constant="${moment_constant}"
+    parent="base_link"
+    mass_rotor="${mass_rotor}"
+    radius_rotor="${radius_rotor}"
+    time_constant="${time_constant}"
+    max_rot_velocity="${max_rot_velocity}"
+    motor_number="2"
+    rotor_drag_coefficient="${rotor_drag_coefficient}"
+    rolling_moment_coefficient="${rolling_moment_coefficient}"
+    color="Red">
+    <origin xyz="${-(arm_length+arm_offset)} 0 ${propeler_offset}" rpy="0 0 0" />
+    <xacro:insert_block name="rotor_inertia" />
+  </xacro:vertical_rotor>
+  <xacro:vertical_rotor
+    robot_namespace="$(arg name)"
+    suffix="right"
+    direction="ccw"
+    motor_constant="${motor_constant}"
+    moment_constant="${moment_constant}"
+    parent="base_link"
+    mass_rotor="${mass_rotor}"
+    radius_rotor="${radius_rotor}"
+    time_constant="${time_constant}"
+    max_rot_velocity="${max_rot_velocity}"
+    motor_number="3"
+    rotor_drag_coefficient="${rotor_drag_coefficient}"
+    rolling_moment_coefficient="${rolling_moment_coefficient}"
+    color="Blue">
+    <origin xyz="0 ${-(arm_length+arm_offset)} ${propeler_offset}" rpy="0 0 0" />
+    <xacro:insert_block name="rotor_inertia" />
+  </xacro:vertical_rotor>
+  <!--xacro:manipulator_left
+    link_length="${link_length}"
+    link_mass="${link_mass}"
+    parent="base_link">
+    <origin xyz="${-(arm_length)} 0 0" rpy="0 0 0" />
+    <xacro:insert_block name="link_inertia"/>
+  </xacro:manipulator_left-->
 </robot>

File: morus_description/urdf/morus.gazebo.xacro (robot description, xacro)
@@ -17,5 +17,5 @@
   <xacro:include filename="$(find morus_description)/urdf/morus.urdf.xacro" />
   <xacro:include filename="$(find rotors_description)/urdf/component_snippets.xacro" />
- <!-- Mount an IMU-->
+ <!-- Mount an IMU - inertial measurement unit-->
   <gazebo>
     <plugin filename="libhector_gazebo_ros_imu.so" name="imu_ros">

File: morus_description/urdf/morus.urdf.xacro (robot description, xacro)
@@ -16,11 +16,11 @@
   <xacro:property name="motor_constant" value="0.000456874" /> <!-- [kg*m/s^2] -->
   <xacro:property name="moment_constant" value="0.01" /> <!-- [m] -->
-  <xacro:property name="time_constant" value="0.125" /> <!-- [s] -->s ti
+  <xacro:property name="time_constant" value="0.125" /> <!-- [s] -->
   <xacro:property name="max_rot_velocity" value="838" /> <!-- [rad/s] -->
   <xacro:property name="rotor_drag_coefficient" value="8.06428e-04" />
   <xacro:property name="rolling_moment_coefficient" value="0.00001" />
-  <xacro:property name="movable_mass_mass" value="1" />
+  <!--xacro:property name="movable_mass_mass" value="1" />
   <xacro:property name="movable_mass_dimension" value="0.08" />
-  <xacro:property name="movable_mass_offset" value="0.025" />
+  <xacro:property name="movable_mass_offset" value="0.025" /-->
   <xacro:property name="imu_mass" value="0.02"/>
   <xacro:property name="imu_size" value="0.01"/>

File: morus_description/urdf/multirotor_base.urdf.xacro (robot description, xacro)
@@ -2,4 +2,13 @@
 <robot xmlns:xacro="http://ros.org/wiki/xacro">
   <!-- Main multirotor link -->
+  <xacro:property name="link_inertia">
+    <inertia
+    ixx="${(link_length * link_mass)/12}"
+    iyy="${(link_length * link_mass)/12}"
+    izz="${(link_length * link_mass)/12}"
+    ixy="0.0" ixz="0.0" iyz="0.0" />
+  </xacro:property>
+  <xacro:property name="link_length" value="0.5" />
+  <xacro:property name="link_mass" value="1" />
   <xacro:macro name="multirotor_base_macro"
     params="robot_namespace mass body_width body_height mesh_file mesh_file_mass *inertia">
@@ -19,7 +28,6 @@
         <origin xyz="0 0 0.125" rpy="0 0 0" />
         <geometry>
-          <mesh filename="package://morus_description/meshes/${mesh_file}"
-            scale="1 1 1" />
-          <!--box size="${body_width} ${body_width} ${body_height}"/--> <!-- [m] [m] [m] -->
+          <!-- mesh filename="package://morus_description/meshes/${mesh_file}" scale="1 1 1" / -->
+          <box size="${body_width} ${body_width} ${body_height}" /> <!-- [m] [m] [m] -->
         </geometry>
       </visual>
@@ -55,4 +63,11 @@
       </plugin>
     </gazebo>
+    <xacro:manipulator_left
+        link_length="${link_length}"
+        link_mass="${link_mass}"
+        parent="base_link">
+        <origin xyz="${-(arm_length)} 0 0" rpy="0 0 0" />
+        <xacro:insert_block name="link_inertia"/>
+    </xacro:manipulator_left>
   </xacro:macro>
   <!-- Macro file for movable mass. It defines joint between mass and stick, and link which defines actual mass. Stick
@@ -70,6 +85,6 @@
     <link name="movable_mass_${mass_number}">
       <visual>
-        <!--origin rpy="0 0 ${orientation}" xyz="0 0 ${0*movable_mass_dimension/2}"/-->
-        <origin rpy="0 0 ${orientation}" xyz="0 0 0"/>
+        <!--origin rpy="0 0 ${orientation}" xyz="0 0 ${0*movable_mass_dimension/2}"/>
+        <origin rpy="0 0 ${orientation}" xyz="0 0 0"/-->
         <geometry>
           <!--mesh filename="package://morus_description/meshes/${mesh_file_mass}"
@@ -114,9 +129,11 @@
       </inertial>
       <visual>
-        <geometry>
-          <!-- <cylinder length="0.005" radius="${radius_rotor}"/> --> <!-- [m] -->
-          <mesh filename="package://morus_description/meshes/propeller_${direction}.dae"
-            scale="0.0025 0.0025 0.0025" />
-          <!-- <box size="${2*radius_rotor} 0.01 0.005"/> -->
+        <!-- origin xyz="10 10 10" rpy="0 0 0" /-->
+        <xacro:insert_block name="origin" />
+        <geometry>
+          <cylinder length="0.005" radius="${radius_rotor}"/> <!-- [m] -->
+          <!--mesh filename="package://morus_description/meshes/propeller_${direction}.dae"
+            scale="0.0025 0.0025 0.0025" /-->
+          <!--box size="${2*radius_rotor} 4 0.005"/-->
         </geometry>
       </visual>
@@ -169,10 +186,10 @@
     </joint>
     <link name="land_gear_${gear_num}">
-      <!--visual>
+      <visual>
         <origin rpy="0 0 0" xyz="0 0 0"/>
         <geometry>
           <box size="0.01 0.01 0.0001"/>
         </geometry>
-      </visual-->
+      </visual>
       <collision>
         <origin rpy="0 0 0" xyz="0 0 0"/>
@@ -255,3 +272,368 @@
     </gazebo>
   </xacro:macro>
+  <!--Spawns left manipulator-->
+  <xacro:macro name="manipulator_left"
+  params="link_length link_mass parent *origin *inertia">
+    <!--link name="link1">
+        <visual>
+            <xacro:insert_block name="origin"/>
+            <geometry>
+                <box size="0.05 0.05 ${link_length}"/>
+            </geometry>
+        </visual>
+        <collision>
+            <xacro:insert_block name="origin"/>
+            <geometry>
+                <box size="0.05 0.05 ${link_length}"/>
+            </geometry>
+        </collision>
+    </link>
+    <link name="link2">
+        <visual>
+            <origin xyz="0 0 -0.25" rpy="-1.57 0 0"/>
+            <geometry>
+                <box size="0.05 0.05 ${link_length}"/>
+            </geometry>
+        </visual>
+        <collision>
+            <origin xyz="0 0 -0.25" rpy="-1.57 0 0"/>
+            <geometry>
+                <box size="0.05 0.05 ${link_length}"/>
+            </geometry>
+        </collision>
+    </link>
+    <joint name="joint_base_link1" type="revolute">
+        <limit upper="3.14" lower="-3.14" effort="0" velocity="0" />
+        <parent link="${parent}"/>
+        <child link="link1"/>
+    </joint>
+    <joint name="joint_link1_link2" type="revolute">
+        <axis xyz="0 1 0"/>
+        <limit upper="3.14" lower="-3.14" effort="0" velocity="0" />
+        <parent link="link1"/>
+        <child link="link2"/>
+        <origin xyz="0 0 -0.25" rpy="-1.57 0 0"/>
+    </joint-->
+    <link name='link1'>
+      <pose frame=''>0 -0.633387 0.200265 0 -0 0</pose>
+      <inertial>
+        <mass value="1" />
+        <xacro:insert_block name="inertia"/>
+        <pose frame=''>0 0 0 0 -0 0</pose>
+      </inertial>
+      <gravity>1</gravity>
+      <self_collide>0</self_collide>
+      <kinematic>0</kinematic>
+      <visual>
+        <pose frame=''>0 0 0 0 -0 0</pose>
+        <geometry>
+           <box size="0.05 0.05 ${link_length}"/>
+        </geometry>
+        <material name="material3">
+          <lighting>1</lighting>
+          <script>
+            <uri>file://media/materials/scripts/gazebo.material</uri>
+            <name>Gazebo/Grey</name>
+          </script>
+          <ambient>0.3 0.3 0.3 1</ambient>
+          <diffuse>0.7 0.7 0.7 1</diffuse>
+          <specular>0.01 0.01 0.01 1</specular>
+          <emissive>0 0 0 1</emissive>
+          <shader type='vertex'>
+            <normal_map>__default__</normal_map>
+          </shader>
+        </material>
+        <cast_shadows>1</cast_shadows>
+        <transparency>0</transparency>
+      </visual>
+      <collision name='collision'>
+        <laser_retro>0</laser_retro>
+        <max_contacts>10</max_contacts>
+        <pose frame=''>0 0 0 0 -0 0</pose>
+        <geometry>
+           <box size="0.05 0.05 ${link_length}"/>
+        </geometry>
+        <surface>
+          <friction>
+            <ode>
+              <mu>1</mu>
+              <mu2>1</mu2>
+              <fdir1>0 0 0</fdir1>
+              <slip1>0</slip1>
+              <slip2>0</slip2>
+            </ode>
+            <torsional>
+              <coefficient>1</coefficient>
+              <patch_radius>0</patch_radius>
+              <surface_radius>0</surface_radius>
+              <use_patch_radius>1</use_patch_radius>
+              <ode>
+                <slip>0</slip>
+              </ode>
+            </torsional>
+          </friction>
+          <bounce>
+            <restitution_coefficient>0</restitution_coefficient>
+            <threshold>1e+06</threshold>
+          </bounce>
+          <contact>
+            <collide_without_contact>0</collide_without_contact>
+            <collide_without_contact_bitmask>1</collide_without_contact_bitmask>
+            <collide_bitmask>1</collide_bitmask>
+            <ode>
+              <soft_cfm>0</soft_cfm>
+              <soft_erp>0.2</soft_erp>
+              <kp>1e+13</kp>
+              <kd>1</kd>
+              <max_vel>0.01</max_vel>
+              <min_depth>0</min_depth>
+            </ode>
+            <bullet>
+              <split_impulse>1</split_impulse>
+              <split_impulse_penetration_threshold>-0.01</split_impulse_penetration_threshold>
+              <soft_cfm>0</soft_cfm>
+              <soft_erp>0.2</soft_erp>
+              <kp>1e+13</kp>
+              <kd>1</kd>
+            </bullet>
+          </contact>
+        </surface>
+      </collision>
+    </link>
+    <link name='link2'>
+      <pose frame=''>0 -0.183347 -0.100133 1.57159 0.001593 3.14159</pose>
+      <inertial>
+        <mass value="1" />
+        <xacro:insert_block name="inertia"/>
+        <pose frame=''>0 0 0 0 -0 0</pose>
+      </inertial>
+      <self_collide>0</self_collide>
+      <kinematic>0</kinematic>
+      <gravity>1</gravity>
+      <visual>
+        <pose frame=''>0 0 0 0 -0 0</pose>
+        <geometry>
+           <box size="0.05 0.05 ${link_length}"/>
+        </geometry>
+        <material name="material2">
+          <lighting>1</lighting>
+          <script>
+            <uri>file://media/materials/scripts/gazebo.material</uri>
+            <name>Gazebo/Grey</name>
+          </script>
+          <ambient>0.3 0.3 0.3 1</ambient>
+          <diffuse>0.7 0.7 0.7 1</diffuse>
+          <specular>0.01 0.01 0.01 1</specular>
+          <emissive>0 0 0 1</emissive>
+          <shader type='vertex'>
+            <normal_map>__default__</normal_map>
+          </shader>
+        </material>
+        <cast_shadows>1</cast_shadows>
+        <transparency>0</transparency>
+      </visual>
+      <collision name='collision'>
+        <laser_retro>0</laser_retro>
+        <max_contacts>10</max_contacts>
+        <pose frame=''>0 0 0 0 -0 0</pose>
+        <geometry>
+           <box size="0.05 0.05 ${link_length}"/>
+        </geometry>
+        <surface>
+          <friction>
+            <ode>
+              <mu>1</mu>
+              <mu2>1</mu2>
+              <fdir1>0 0 0</fdir1>
+              <slip1>0</slip1>
+              <slip2>0</slip2>
+            </ode>
+            <torsional>
+              <coefficient>1</coefficient>
+              <patch_radius>0</patch_radius>
+              <surface_radius>0</surface_radius>
+              <use_patch_radius>1</use_patch_radius>
+              <ode>
+                <slip>0</slip>
+              </ode>
+            </torsional>
+          </friction>
+          <bounce>
+            <restitution_coefficient>0</restitution_coefficient>
+            <threshold>1e+06</threshold>
+          </bounce>
+          <contact>
+            <collide_without_contact>0</collide_without_contact>
+            <collide_without_contact_bitmask>1</collide_without_contact_bitmask>
+            <collide_bitmask>1</collide_bitmask>
+            <ode>
+              <soft_cfm>0</soft_cfm>
+              <soft_erp>0.2</soft_erp>
+              <kp>1e+13</kp>
+              <kd>1</kd>
+              <max_vel>0.01</max_vel>
+              <min_depth>0</min_depth>
+            </ode>
+            <bullet>
+              <split_impulse>1</split_impulse>
+              <split_impulse_penetration_threshold>-0.01</split_impulse_penetration_threshold>
+              <soft_cfm>0</soft_cfm>
+              <soft_erp>0.2</soft_erp>
+              <kp>1e+13</kp>
+              <kd>1</kd>
+            </bullet>
+          </contact>
+        </surface>
+      </collision>
+    </link>
+    <link name='link3'>
+      <pose frame=''>0 0.816733 -0.100133 1.57159 0.001593 3.14159</pose>
+      <inertial>
+        <mass value="1"/>
+        <xacro:insert_block name="inertia"/>
+        <pose frame=''>0 0 0 0 -0 0</pose>
+      </inertial>
+      <self_collide>0</self_collide>
+      <kinematic>0</kinematic>
+      <gravity>1</gravity>
+      <visual>
+        <pose frame=''>0 0 0 0 -0 0</pose>
+        <geometry>
+           <box size="0.05 0.05 ${link_length}"/>
+        </geometry>
+        <material name="material1">
+          <lighting>1</lighting>
+          <script>
+            <uri>file://media/materials/scripts/gazebo.material</uri>
+            <name>Gazebo/Grey</name>
+          </script>
+          <ambient>0.3 0.3 0.3 1</ambient>
+          <diffuse>0.7 0.7 0.7 1</diffuse>
+          <specular>0.01 0.01 0.01 1</specular>
+          <emissive>0 0 0 1</emissive>
+          <shader type='vertex'>
+            <normal_map>__default__</normal_map>
+          </shader>
+        </material>
+        <cast_shadows>1</cast_shadows>
+        <transparency>0</transparency>
+      </visual>
+      <collision name='collision'>
+        <laser_retro>0</laser_retro>
+        <max_contacts>10</max_contacts>
+        <pose frame=''>0 0 0 0 -0 0</pose>
+        <geometry>
+           <box size="0.05 0.05 ${link_length}"/>
+        </geometry>
+        <surface>
+          <friction>
+            <ode>
+              <mu>1</mu>
+              <mu2>1</mu2>
+              <fdir1>0 0 0</fdir1>
+              <slip1>0</slip1>
+              <slip2>0</slip2>
+            </ode>
+            <torsional>
+              <coefficient>1</coefficient>
+              <patch_radius>0</patch_radius>
+              <surface_radius>0</surface_radius>
+              <use_patch_radius>1</use_patch_radius>
+              <ode>
+                <slip>0</slip>
+              </ode>
+            </torsional>
+          </friction>
+          <bounce>
+            <restitution_coefficient>0</restitution_coefficient>
+            <threshold>1e+06</threshold>
+          </bounce>
+          <contact>
+            <collide_without_contact>0</collide_without_contact>
+            <collide_without_contact_bitmask>1</collide_without_contact_bitmask>
+            <collide_bitmask>1</collide_bitmask>
+            <ode>
+              <soft_cfm>0</soft_cfm>
+              <soft_erp>0.2</soft_erp>
+              <kp>1e+13</kp>
+              <kd>1</kd>
+              <max_vel>0.01</max_vel>
+              <min_depth>0</min_depth>
+            </ode>
+            <bullet>
+              <split_impulse>1</split_impulse>
+              <split_impulse_penetration_threshold>-0.01</split_impulse_penetration_threshold>
+              <soft_cfm>0</soft_cfm>
+              <soft_erp>0.2</soft_erp>
+              <kp>1e+13</kp>
+              <kd>1</kd>
+            </bullet>
+          </contact>
+        </surface>
+      </collision>
+    </link>
+    <joint name="joint_base_link1" type="fixed">
+        <xacro:insert_block name="origin"/>
+        <parent link="${parent}"/>
+        <child link="link1"/>
+    </joint>
+    <joint name='joint_link1_link2' type='revolute'>
+      <parent link="link1" />
+      <child link="link2" />
+      <pose frame=''>0 0 -0.5 0 -0 0</pose>
+      <limit upper="1.79769e+308" lower="-1.79769e+308" effort="-1" velocity="-1" />
+      <axis>
+        <xyz>0 1 0</xyz>
+        <use_parent_model_frame>0</use_parent_model_frame>
+        <dynamics>
+          <spring_reference>0</spring_reference>
+          <spring_stiffness>0</spring_stiffness>
+          <damping>0</damping>
+          <friction>0</friction>
+        </dynamics>
+      </axis>
+      <physics>
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