Commit message: Add double manipulator

File: morus_description/urdf/morus.base.urdf.xacro (robot description, xacro)
@@ -178,10 +178,19 @@
     <xacro:insert_block name="rotor_inertia" />
   </xacro:vertical_rotor>
-  <!--xacro:manipulator_left
+  <xacro:manipulator
     link_length="${link_length}"
     link_mass="${link_mass}"
-    parent="base_link">
-    <origin xyz="${-(arm_length)} 0 0" rpy="0 0 0" />
+    parent="base_link"
+    suffix="left">
+    <origin xyz="${-(arm_length)} 0 ${-(link_length/2)}" rpy="0 0 0" />
     <xacro:insert_block name="link_inertia"/>
-  </xacro:manipulator_left-->
+  </xacro:manipulator>
+  <xacro:manipulator
+    link_length="${link_length}"
+    link_mass="${link_mass}"
+    parent="base_link"
+    suffix="right">
+    <origin xyz="${arm_length} 0 ${-(link_length/2)}" rpy="0 0 0" />
+    <xacro:insert_block name="link_inertia"/>
+  </xacro:manipulator>
 </robot>

File: morus_description/urdf/multirotor_base.urdf.xacro (robot description, xacro)
@@ -63,11 +63,4 @@
       </plugin>
     </gazebo>
-    <xacro:manipulator_left
-        link_length="${link_length}"
-        link_mass="${link_mass}"
-        parent="base_link">
-        <origin xyz="${-(arm_length)} 0 0" rpy="0 0 0" />
-        <xacro:insert_block name="link_inertia"/>
-    </xacro:manipulator_left>
   </xacro:macro>
   <!-- Macro file for movable mass. It defines joint between mass and stick, and link which defines actual mass. Stick
@@ -272,49 +265,47 @@
     </gazebo>
   </xacro:macro>
-  <!--Spawns left manipulator-->
-  <xacro:macro name="manipulator_left"
-  params="link_length link_mass parent *origin *inertia">
-    <!--link name="link1">
-        <visual>
-            <xacro:insert_block name="origin"/>
-            <geometry>
-                <box size="0.05 0.05 ${link_length}"/>
-            </geometry>
-        </visual>
-        <collision>
-            <xacro:insert_block name="origin"/>
-            <geometry>
-                <box size="0.05 0.05 ${link_length}"/>
-            </geometry>
-        </collision>
-    </link>
-    <link name="link2">
-        <visual>
-            <origin xyz="0 0 -0.25" rpy="-1.57 0 0"/>
-            <geometry>
-                <box size="0.05 0.05 ${link_length}"/>
-            </geometry>
-        </visual>
-        <collision>
-            <origin xyz="0 0 -0.25" rpy="-1.57 0 0"/>
-            <geometry>
-                <box size="0.05 0.05 ${link_length}"/>
-            </geometry>
-        </collision>
-    </link>
-    <joint name="joint_base_link1" type="revolute">
-        <limit upper="3.14" lower="-3.14" effort="0" velocity="0" />
-        <parent link="${parent}"/>
-        <child link="link1"/>
-    </joint>
-    <joint name="joint_link1_link2" type="revolute">
-        <axis xyz="0 1 0"/>
-        <limit upper="3.14" lower="-3.14" effort="0" velocity="0" />
-        <parent link="link1"/>
-        <child link="link2"/>
-        <origin xyz="0 0 -0.25" rpy="-1.57 0 0"/>
-    </joint-->
-    <link name='link1'>
-      <pose frame=''>0 -0.633387 0.200265 0 -0 0</pose>
+  <!--Spawns left manipulator:
+  Manipulator is modeled as a 2DOF manipulator where first link is
+  fixed to the base. Other two links are conecteted with
+  revolute joints -->
+  <!--macro arguments -
+  - link length
+  - link mass
+  - parent of the first (fixed) link
+  - origin block determining position of the first link
+  - intertial block definining link inertia
+  -->
+  <xacro:macro name="manipulator"
+  params="link_length link_mass parent suffix *origin *inertia">
+    <!--_____________________________________________________________-->
+    <!--LINK1-->
+    <!--_____________________________________________________________-->
+    <link name='link_fixed_${suffix}'>
+      <origin xyz="0 0 0" rpy="0 0 0"/>
+      <inertial>
+        <mass value="1" />
+        <xacro:insert_block name="inertia"/>
+        <pose xyz="0 0 0" rpy="0 0 0"/>
+      </inertial>
+      <visual>
+        <geometry>
+           <box size="0.05 0.05 ${link_length/2}"/>
+        </geometry>
+      </visual>
+      <collision name='collision'>
+        <origin xyz="0 0 0" rpy="0 0 0"/>
+        <geometry>
+           <box size="0.05 0.05 ${link_length/2}"/>
+        </geometry>
+      </collision>
+    </link>
+    <gazebo reference="link_fixed_${suffix}">
+      <material>Gazebo/Red</material>
+    </gazebo>
+    <!--_____________________________________________________________-->
+    <!--LINK2-->
+    <!--_____________________________________________________________-->
+    <link name='link_middle_${suffix}'>
+      <origin xyz="0 0 0" rpy="0 0 0"/>
       <inertial>
         <mass value="1" />
@@ -322,7 +313,7 @@
         <pose frame=''>0 0 0 0 -0 0</pose>
       </inertial>
-      <gravity>1</gravity>
       <self_collide>0</self_collide>
       <kinematic>0</kinematic>
+      <gravity>1</gravity>
       <visual>
         <pose frame=''>0 0 0 0 -0 0</pose>
@@ -330,9 +321,9 @@
            <box size="0.05 0.05 ${link_length}"/>
         </geometry>
-        <material name="material3">
+        <material name="material2">
           <lighting>1</lighting>
           <script>
             <uri>file://media/materials/scripts/gazebo.material</uri>
-            <name>Gazebo/Grey</name>
+            <name>Gazebo/Blue</name>
           </script>
           <ambient>0.3 0.3 0.3 1</ambient>
@@ -401,8 +392,14 @@
       </collision>
     </link>
-    <link name='link2'>
-      <pose frame=''>0 -0.183347 -0.100133 1.57159 0.001593 3.14159</pose>
-      <inertial>
-        <mass value="1" />
+    <gazebo reference="link_middle_${suffix}">
+      <material>Gazebo/Blue</material>
+    </gazebo>
+    <!--_____________________________________________________________-->
+    <!--LINK3-->
+    <!--_____________________________________________________________-->
+    <link name='link_end_${suffix}'>
+      <pose frame=''>0 0.816733 -0.100133 1.57159 0.001593 3.14159</pose>
+      <inertial>
+        <mass value="1"/>
         <xacro:insert_block name="inertia"/>
         <pose frame=''>0 0 0 0 -0 0</pose>
@@ -416,9 +413,9 @@
            <box size="0.05 0.05 ${link_length}"/>
         </geometry>
-        <material name="material2">
+        <material name="material1">
           <lighting>1</lighting>
           <script>
             <uri>file://media/materials/scripts/gazebo.material</uri>
-            <name>Gazebo/Grey</name>
+            <name>Gazebo/Green</name>
           </script>
           <ambient>0.3 0.3 0.3 1</ambient>
@@ -487,99 +484,24 @@
       </collision>
     </link>
-    <link name='link3'>
-      <pose frame=''>0 0.816733 -0.100133 1.57159 0.001593 3.14159</pose>
-      <inertial>
-        <mass value="1"/>
-        <xacro:insert_block name="inertia"/>
-        <pose frame=''>0 0 0 0 -0 0</pose>
-      </inertial>
-      <self_collide>0</self_collide>
-      <kinematic>0</kinematic>
-      <gravity>1</gravity>
-      <visual>
-        <pose frame=''>0 0 0 0 -0 0</pose>
-        <geometry>
-           <box size="0.05 0.05 ${link_length}"/>
-        </geometry>
-        <material name="material1">
-          <lighting>1</lighting>
-          <script>
-            <uri>file://media/materials/scripts/gazebo.material</uri>
-            <name>Gazebo/Grey</name>
-          </script>
-          <ambient>0.3 0.3 0.3 1</ambient>
-          <diffuse>0.7 0.7 0.7 1</diffuse>
-          <specular>0.01 0.01 0.01 1</specular>
-          <emissive>0 0 0 1</emissive>
-          <shader type='vertex'>
-            <normal_map>__default__</normal_map>
-          </shader>
-        </material>
-        <cast_shadows>1</cast_shadows>
-        <transparency>0</transparency>
-      </visual>
-      <collision name='collision'>
-        <laser_retro>0</laser_retro>
-        <max_contacts>10</max_contacts>
-        <pose frame=''>0 0 0 0 -0 0</pose>
-        <geometry>
-           <box size="0.05 0.05 ${link_length}"/>
-        </geometry>
-        <surface>
-          <friction>
-            <ode>
-              <mu>1</mu>
-              <mu2>1</mu2>
-              <fdir1>0 0 0</fdir1>
-              <slip1>0</slip1>
-              <slip2>0</slip2>
-            </ode>
-            <torsional>
-              <coefficient>1</coefficient>
-              <patch_radius>0</patch_radius>
-              <surface_radius>0</surface_radius>
-              <use_patch_radius>1</use_patch_radius>
-              <ode>
-                <slip>0</slip>
-              </ode>
-            </torsional>
-          </friction>
-          <bounce>
-            <restitution_coefficient>0</restitution_coefficient>
-            <threshold>1e+06</threshold>
-          </bounce>
-          <contact>
-            <collide_without_contact>0</collide_without_contact>
-            <collide_without_contact_bitmask>1</collide_without_contact_bitmask>
-            <collide_bitmask>1</collide_bitmask>
-            <ode>
-              <soft_cfm>0</soft_cfm>
-              <soft_erp>0.2</soft_erp>
-              <kp>1e+13</kp>
-              <kd>1</kd>
-              <max_vel>0.01</max_vel>
-              <min_depth>0</min_depth>
-            </ode>
-            <bullet>
-              <split_impulse>1</split_impulse>
-              <split_impulse_penetration_threshold>-0.01</split_impulse_penetration_threshold>
-              <soft_cfm>0</soft_cfm>
-              <soft_erp>0.2</soft_erp>
-              <kp>1e+13</kp>
-              <kd>1</kd>
-            </bullet>
-          </contact>
-        </surface>
-      </collision>
-    </link>
-    <joint name="joint_base_link1" type="fixed">
+    <gazebo reference="link_end_${suffix}">
+      <material>Gazebo/Green</material>
+    </gazebo>
+    <!--_____________________________________________________________-->
+    <!--JOINT_baseToFixed-->
+    <!--Fixed joint connecting base to first link (fixed)-->
+    <!--_____________________________________________________________-->
+    <joint name="joint_baseToFixed_${suffix}" type="fixed">
         <xacro:insert_block name="origin"/>
         <parent link="${parent}"/>
-        <child link="link1"/>
-    </joint>
-    <joint name='joint_link1_link2' type='revolute'>
-      <parent link="link1" />
-      <child link="link2" />
-      <pose frame=''>0 0 -0.5 0 -0 0</pose>
+        <child link="link_fixed_${suffix}"/>
+    </joint>
+    <!--_____________________________________________________________-->
+    <!--JOINT_fixedtoMiddle-->
+    <!--Revolute joint connecting fixed link to middle link-->
+    <!--_____________________________________________________________-->
+    <joint name='joint_fixedToMiddle_${suffix}' type='revolute'>
+      <parent link="link_fixed_${suffix}" />
+      <child link="link_middle_${suffix}" />
+      <origin xyz="0 -0.183347 -0.100133" rpy="1.57159 0.00 3.14159"/>
       <limit upper="1.79769e+308" lower="-1.79769e+308" effort="-1" velocity="-1" />
       <axis>
@@ -606,8 +528,12 @@
       </physics>
     </joint>
-    <joint name="joint_link2_link3" type="revolute">
-      <parent link="link2" />
-      <child link="link3" />
-      <pose frame=''>0 0 -0.5 0 -0 0</pose>
+    <!--_____________________________________________________________-->
+    <!--JOINT_middleToEnd-->
+    <!--Revolute joint connecting middle link to end link.-->
+    <!--_____________________________________________________________-->
+    <joint name="joint_middleToEnd_${suffix}" type="revolute">
+      <parent link="link_middle_${suffix}" />
+      <child link="link_end_${suffix}" />
+      <origin xyz="0 0 ${-link_length}" rpy="0 0 0"/>
       <limit upper="1.79769e+308" lower="-1.79769e+308" effort="-1" velocity="-1" />
       <axis>
