Commit message: Fix coordinate system

File: morus_description/urdf/morus.base.gazebo.xacro (robot description, xacro)
@@ -21,5 +21,5 @@
       <robotNamespace>$(arg name)</robotNamespace>
       <imuTopicName>/morus/ahrs</imuTopicName>
-      <connectedICEs>/morus/gm_back_status /morus/gm_front_status /morus/gm_left_status /morus/gm_right_status /morus/collectiveThrust</connectedICEs>
+      <connectedICEs>/morus/gm_back_status /morus/gm_front_status /morus_descriptions/gm_left_status /morus/gm_right_status /morus/collectiveThrust</connectedICEs>
     </plugin>
   </gazebo>

File: morus_description/urdf/morus.base.urdf.xacro (robot description, xacro)
@@ -31,4 +31,5 @@
   <xacro:property name="link_length" value="0.5" />
   <xacro:property name="link_mass" value="1" />
+  <xacro:property name="link_width" value="0.05" />
   <!-- Property Blocks -->
   <xacro:property name="body_inertia">
@@ -178,6 +179,8 @@
     <xacro:insert_block name="rotor_inertia" />
   </xacro:vertical_rotor>
+  <!-- Adding left manipulator -->
   <xacro:manipulator
     link_length="${link_length}"
+    link_width="${link_width}"
     link_mass="${link_mass}"
     parent="base_link"
@@ -186,6 +189,8 @@
     <xacro:insert_block name="link_inertia"/>
   </xacro:manipulator>
+  <!-- Adding right manipulator -->
   <xacro:manipulator
     link_length="${link_length}"
+    link_width="${link_width}"
     link_mass="${link_mass}"
     parent="base_link"

File: morus_description/urdf/multirotor_base.urdf.xacro (robot description, xacro)
@@ -9,4 +9,5 @@
     ixy="0.0" ixz="0.0" iyz="0.0" />
   </xacro:property>
+  <xacro:property name="PI" value="3.14" />
   <xacro:property name="link_length" value="0.5" />
   <xacro:property name="link_mass" value="1" />
@@ -265,5 +266,5 @@
     </gazebo>
   </xacro:macro>
-  <!--Spawns left manipulator:
+  <!--Spawns manipulator:
   Manipulator is modeled as a 2DOF manipulator where first link is
   fixed to the base. Other two links are conecteted with
@@ -277,5 +278,5 @@
   -->
   <xacro:macro name="manipulator"
-  params="link_length link_mass parent suffix *origin *inertia">
+  params="link_length link_width link_mass parent suffix *origin *inertia">
     <!--_____________________________________________________________-->
     <!--LINK1-->
@@ -290,5 +291,5 @@
       <visual>
         <geometry>
-           <box size="0.05 0.05 ${link_length/2}"/>
+           <box size="${link_width} ${link_width} ${link_length/2}"/>
         </geometry>
       </visual>
@@ -296,5 +297,5 @@
         <origin xyz="0 0 0" rpy="0 0 0"/>
         <geometry>
-           <box size="0.05 0.05 ${link_length/2}"/>
+           <box size="${link_width} ${link_width} ${link_length/2}"/>
         </geometry>
       </collision>
@@ -307,87 +308,20 @@
     <!--_____________________________________________________________-->
     <link name='link_middle_${suffix}'>
-      <origin xyz="0 0 0" rpy="0 0 0"/>
       <inertial>
         <mass value="1" />
         <xacro:insert_block name="inertia"/>
-        <pose frame=''>0 0 0 0 -0 0</pose>
-      </inertial>
-      <self_collide>0</self_collide>
-      <kinematic>0</kinematic>
-      <gravity>1</gravity>
-      <visual>
-        <pose frame=''>0 0 0 0 -0 0</pose>
-        <geometry>
-           <box size="0.05 0.05 ${link_length}"/>
-        </geometry>
-        <material name="material2">
-          <lighting>1</lighting>
-          <script>
-            <uri>file://media/materials/scripts/gazebo.material</uri>
-            <name>Gazebo/Blue</name>
-          </script>
-          <ambient>0.3 0.3 0.3 1</ambient>
-          <diffuse>0.7 0.7 0.7 1</diffuse>
-          <specular>0.01 0.01 0.01 1</specular>
-          <emissive>0 0 0 1</emissive>
-          <shader type='vertex'>
-            <normal_map>__default__</normal_map>
-          </shader>
-        </material>
-        <cast_shadows>1</cast_shadows>
-        <transparency>0</transparency>
-      </visual>
+        <origin xyz="0 0 0" rpy="0 0 0"/>
+      </inertial>
+      <visual>
+        <origin rpy="0 0 0" xyz="0 ${-link_length/2 + link_width/2} 0"/>
+        <geometry>
+           <box size="${link_width} ${link_length} ${link_width}"/>
+        </geometry>
+     </visual>
       <collision name='collision'>
-        <laser_retro>0</laser_retro>
-        <max_contacts>10</max_contacts>
-        <pose frame=''>0 0 0 0 -0 0</pose>
-        <geometry>
-           <box size="0.05 0.05 ${link_length}"/>
-        </geometry>
-        <surface>
-          <friction>
-            <ode>
-              <mu>1</mu>
-              <mu2>1</mu2>
-              <fdir1>0 0 0</fdir1>
-              <slip1>0</slip1>
-              <slip2>0</slip2>
-            </ode>
-            <torsional>
-              <coefficient>1</coefficient>
-              <patch_radius>0</patch_radius>
-              <surface_radius>0</surface_radius>
-              <use_patch_radius>1</use_patch_radius>
-              <ode>
-                <slip>0</slip>
-              </ode>
-            </torsional>
-          </friction>
-          <bounce>
-            <restitution_coefficient>0</restitution_coefficient>
-            <threshold>1e+06</threshold>
-          </bounce>
-          <contact>
-            <collide_without_contact>0</collide_without_contact>
-            <collide_without_contact_bitmask>1</collide_without_contact_bitmask>
-            <collide_bitmask>1</collide_bitmask>
-            <ode>
-              <soft_cfm>0</soft_cfm>
-              <soft_erp>0.2</soft_erp>
-              <kp>1e+13</kp>
-              <kd>1</kd>
-              <max_vel>0.01</max_vel>
-              <min_depth>0</min_depth>
-            </ode>
-            <bullet>
-              <split_impulse>1</split_impulse>
-              <split_impulse_penetration_threshold>-0.01</split_impulse_penetration_threshold>
-              <soft_cfm>0</soft_cfm>
-              <soft_erp>0.2</soft_erp>
-              <kp>1e+13</kp>
-              <kd>1</kd>
-            </bullet>
-          </contact>
-        </surface>
+        <origin rpy="0 0 0" xyz="0 ${-link_length/2 + link_width/2} 0"/>
+        <geometry>
+           <box size="${link_length} ${link_width} ${link_width}"/>
+        </geometry>
       </collision>
     </link>
@@ -399,87 +333,20 @@
     <!--_____________________________________________________________-->
     <link name='link_end_${suffix}'>
-      <pose frame=''>0 0.816733 -0.100133 1.57159 0.001593 3.14159</pose>
       <inertial>
         <mass value="1"/>
         <xacro:insert_block name="inertia"/>
-        <pose frame=''>0 0 0 0 -0 0</pose>
-      </inertial>
-      <self_collide>0</self_collide>
-      <kinematic>0</kinematic>
-      <gravity>1</gravity>
-      <visual>
-        <pose frame=''>0 0 0 0 -0 0</pose>
-        <geometry>
-           <box size="0.05 0.05 ${link_length}"/>
-        </geometry>
-        <material name="material1">
-          <lighting>1</lighting>
-          <script>
-            <uri>file://media/materials/scripts/gazebo.material</uri>
-            <name>Gazebo/Green</name>
-          </script>
-          <ambient>0.3 0.3 0.3 1</ambient>
-          <diffuse>0.7 0.7 0.7 1</diffuse>
-          <specular>0.01 0.01 0.01 1</specular>
-          <emissive>0 0 0 1</emissive>
-          <shader type='vertex'>
-            <normal_map>__default__</normal_map>
-          </shader>
-        </material>
-        <cast_shadows>1</cast_shadows>
-        <transparency>0</transparency>
+        <origin xyz="0 0 0" rpy="0 0 0"/>
+      </inertial>
+      <visual>
+        <origin xyz="0 ${-link_length/2} 0" rpy="0 0 0"/>
+        <geometry>
+           <box size="${link_width} ${link_length} ${link_width}"/>
+        </geometry>
       </visual>
       <collision name='collision'>
-        <laser_retro>0</laser_retro>
-        <max_contacts>10</max_contacts>
-        <pose frame=''>0 0 0 0 -0 0</pose>
-        <geometry>
-           <box size="0.05 0.05 ${link_length}"/>
-        </geometry>
-        <surface>
-          <friction>
-            <ode>
-              <mu>1</mu>
-              <mu2>1</mu2>
-              <fdir1>0 0 0</fdir1>
-              <slip1>0</slip1>
-              <slip2>0</slip2>
-            </ode>
-            <torsional>
-              <coefficient>1</coefficient>
-              <patch_radius>0</patch_radius>
-              <surface_radius>0</surface_radius>
-              <use_patch_radius>1</use_patch_radius>
-              <ode>
-                <slip>0</slip>
-              </ode>
-            </torsional>
-          </friction>
-          <bounce>
-            <restitution_coefficient>0</restitution_coefficient>
-            <threshold>1e+06</threshold>
-          </bounce>
-          <contact>
-            <collide_without_contact>0</collide_without_contact>
-            <collide_without_contact_bitmask>1</collide_without_contact_bitmask>
-            <collide_bitmask>1</collide_bitmask>
-            <ode>
-              <soft_cfm>0</soft_cfm>
-              <soft_erp>0.2</soft_erp>
-              <kp>1e+13</kp>
-              <kd>1</kd>
-              <max_vel>0.01</max_vel>
-              <min_depth>0</min_depth>
-            </ode>
-            <bullet>
-              <split_impulse>1</split_impulse>
-              <split_impulse_penetration_threshold>-0.01</split_impulse_penetration_threshold>
-              <soft_cfm>0</soft_cfm>
-              <soft_erp>0.2</soft_erp>
-              <kp>1e+13</kp>
-              <kd>1</kd>
-            </bullet>
-          </contact>
-        </surface>
+        <origin xyz="0 ${-link_length/2} 0" rpy="0 0 0"/>
+        <geometry>
+           <box size="${link_width} ${link_length} ${link_width}"/>
+        </geometry>
       </collision>
     </link>
@@ -503,8 +370,8 @@
       <parent link="link_fixed_${suffix}" />
       <child link="link_middle_${suffix}" />
-      <origin xyz="0 -0.183347 -0.100133" rpy="1.57159 0.00 3.14159"/>
-      <limit upper="1.79769e+308" lower="-1.79769e+308" effort="-1" velocity="-1" />
+      <origin xyz="0 0 ${-(link_length/4 + link_width/2)}" rpy="0 0 0"/>
+      <limit upper="1.79769e+308" lower="-1.79769e+308" effort="-1" velocity="-1"/>
       <axis>
-        <xyz>0 1 0</xyz>
+        <xyz>0 0 1</xyz>
         <use_parent_model_frame>0</use_parent_model_frame>
         <dynamics>
@@ -535,8 +402,8 @@
       <parent link="link_middle_${suffix}" />
       <child link="link_end_${suffix}" />
-      <origin xyz="0 0 ${-link_length}" rpy="0 0 0"/>
+      <origin xyz="0 ${-link_length} 0" rpy="0 0 0"/>
       <limit upper="1.79769e+308" lower="-1.79769e+308" effort="-1" velocity="-1" />
       <axis>
-        <xyz>0 1 0</xyz>
+        <xyz>0 0 1</xyz>
         <use_parent_model_frame>0</use_parent_model_frame>
         <dynamics>
@@ -560,6 +427,4 @@
       </physics>
     </joint>
-    <static>0</static>
-    <allow_auto_disable>1</allow_auto_disable>
   </xacro:macro>
 </robot>

Commit message: Add control, not working

File: morus_description/urdf/morus.base.gazebo.xacro (robot description, xacro)
@@ -8,4 +8,6 @@
     <plugin name="gazebo_ros_control" filename="libgazebo_ros_control.so">
       <robotNamespace>/morus</robotNamespace>
+       <!-- Added robot description -->
+       <robotParam>/morus/robot_description </robotParam>
        <robotSimType>gazebo_ros_control/DefaultRobotHWSim</robotSimType>
     </plugin>

File: morus_description/urdf/morus.base.urdf.xacro (robot description, xacro)
@@ -199,3 +199,20 @@
     <xacro:insert_block name="link_inertia"/>
   </xacro:manipulator>
+  <!-- Add transmission for joints -->
+  <xacro:transmisija
+    trans_number="0"
+    joint_name="joint_baseToFixed_left">
+  </xacro:transmisija>
+  <xacro:transmisija
+    trans_number="1"
+    joint_name="joint_middleToEnd_left">
+  </xacro:transmisija>
+  <xacro:transmisija
+    trans_number="2"
+    joint_name="joint_baseToFixed_right">
+  </xacro:transmisija>
+  <xacro:transmisija
+    trans_number="3"
+    joint_name="joint_middleToEnd_right">
+  </xacro:transmisija>
 </robot>

File: morus_description/urdf/morus.urdf.xacro (robot description, xacro)
@@ -20,7 +20,7 @@
   <xacro:property name="rotor_drag_coefficient" value="8.06428e-04" />
   <xacro:property name="rolling_moment_coefficient" value="0.00001" />
-  <!--xacro:property name="movable_mass_mass" value="1" />
+  <xacro:property name="movable_mass_mass" value="1" />
   <xacro:property name="movable_mass_dimension" value="0.08" />
-  <xacro:property name="movable_mass_offset" value="0.025" /-->
+  <xacro:property name="movable_mass_offset" value="0.025" />
   <xacro:property name="imu_mass" value="0.02"/>
   <xacro:property name="imu_size" value="0.01"/>
@@ -56,4 +56,15 @@
     ixy="0.0" ixz="0.0"  iyz="0.0" /> <!-- [kg*m^2] [kg*m^2] [kg*m^2] [kg*m^2] [kg*m^2] [kg*m^2] -->
   </xacro:property>
+  <!-- Manipulator properties-->
+  <xacro:property name="link_length" value="0.5" />
+  <xacro:property name="link_mass" value="1" />
+  <xacro:property name="link_width" value="0.05" />
+  <xacro:property name="link_inertia">
+    <inertia
+    ixx="${(link_length * link_mass)/12}"
+    iyy="${(link_length * link_mass)/12}"
+    izz="${(link_length * link_mass)/12}"
+    ixy="0.0" ixz="0.0" iyz="0.0" />
+  </xacro:property>
   <!-- Included URDF Files -->
   <xacro:include filename="$(find morus_description)/urdf/multirotor_base.urdf.xacro" />
@@ -142,5 +153,5 @@
   </xacro:vertical_rotor>
   <!-- Instantiate movable mass 0-->
-  <xacro:movable_mass
+  <!--xacro:movable_mass
     mass_number="0"
     parent="base_link"
@@ -154,7 +165,7 @@
     <origin xyz="${(arm_length/2+arm_offset)} 0.0 ${movable_mass_offset}" rpy="0 0 0" />
     <xacro:insert_block name="movable_mass_inertia"/>
-  </xacro:movable_mass>
+  </xacro:movable_mass-->
   <!-- Instantiate movable mass 1 -->
-  <xacro:movable_mass
+  <!--xacro:movable_mass
     mass_number="1"
     parent="base_link"
@@ -168,7 +179,7 @@
     <origin xyz="0.0 ${(arm_length/2+arm_offset)} ${movable_mass_offset}" rpy="0 0 0" />
     <xacro:insert_block name="movable_mass_inertia"/>
-  </xacro:movable_mass>
+  </xacro:movable_mass-->
   <!-- Instantiate movable mass 2-->
-  <xacro:movable_mass
+  <!--xacro:movable_mass
     mass_number="2"
     parent="base_link"
@@ -182,7 +193,7 @@
     <origin xyz="${-(arm_length/2+arm_offset)} 0.0 ${movable_mass_offset}" rpy="0 0 0" />
     <xacro:insert_block name="movable_mass_inertia"/>
-  </xacro:movable_mass>
+  </xacro:movable_mass-->
   <!-- Instantiate movable mass 3 -->
-  <xacro:movable_mass
+  <!--xacro:movable_mass
     mass_number="3"
     parent="base_link"
@@ -196,6 +207,6 @@
     <origin xyz="0.0 ${-(arm_length/2+arm_offset)} ${movable_mass_offset}" rpy="0 0 0" />
     <xacro:insert_block name="movable_mass_inertia"/>
-  </xacro:movable_mass>
-  <xacro:transmisija
+  </xacro:movable_mass-->
+  <!--xacro:transmisija
     trans_number="0"
     joint_name="stick_to_movable_mass_0">
@@ -212,5 +223,5 @@
     trans_number="3"
     joint_name="stick_to_movable_mass_3">
-  </xacro:transmisija>
+  </xacro:transmisija-->
   <xacro:property name="land_gear_inertia">
     <inertia
@@ -240,3 +251,23 @@
       <xacro:insert_block name="land_gear_inertia"/>
   </xacro:landing_gear>
+   <!-- Adding left manipulator -->
+  <xacro:manipulator
+    link_length="${link_length}"
+    link_width="${link_width}"
+    link_mass="${link_mass}"
+    parent="base_link"
+    suffix="left">
+    <origin xyz="${-(arm_length)} 0 ${-(link_length/2)}" rpy="0 0 0" />
+    <xacro:insert_block name="link_inertia"/>
+  </xacro:manipulator>
+  <!-- Adding right manipulator -->
+  <xacro:manipulator
+    link_length="${link_length}"
+    link_width="${link_width}"
+    link_mass="${link_mass}"
+    parent="base_link"
+    suffix="right">
+    <origin xyz="${arm_length} 0 ${-(link_length/2)}" rpy="0 0 0" />
+    <xacro:insert_block name="link_inertia"/>
+  </xacro:manipulator>
 </robot>

Commit message: Added manipulator_ctl_attitude.py

File: morus_description/urdf/morus.base.gazebo.xacro (robot description, xacro)
@@ -8,6 +8,6 @@
     <plugin name="gazebo_ros_control" filename="libgazebo_ros_control.so">
       <robotNamespace>/morus</robotNamespace>
-       <!-- Added robot description -->
-       <robotParam>/morus/robot_description </robotParam>
+       <!-- Added robot description <name /-->
+       <robotParam>/morus/robot_description</robotParam>
        <robotSimType>gazebo_ros_control/DefaultRobotHWSim</robotSimType>
     </plugin>
@@ -18,4 +18,25 @@
   <xacro:include filename="$(find morus_description)/urdf/morus.base.urdf.xacro" />
   <xacro:include filename="$(find rotors_description)/urdf/component_snippets.xacro" />
+  <!-- Mount an IMU - inertial measurement unit-->
+  <gazebo>
+    <plugin filename="libhector_gazebo_ros_imu.so" name="imu_ros">
+      <robotNamespace>$(arg name)</robotNamespace>
+      <bodyName>base_link</bodyName> <!-- (string, required): name of the body which holds the IMU sensor -->
+      <topicName>imu</topicName> <!-- (string): name of the sensor output topic and prefix of service names (defaults to imu) -->
+      <accelOffset>0.0 0.0 0.0</accelOffset> <!-- (Vector3): constant acceleration offset -->
+      <accelDrift>0.0 0.0 0.0</accelDrift> <!-- (Vector3): standard deviation of the acceleration drift error -->
+      <accelDriftFrequency>0.0 0.0 0.0</accelDriftFrequency> <!-- (Vector3): mean frequency of the acceleration drift staviti na nulu-->
+      <accelGaussianNoise>0.0 0.0 0.0</accelGaussianNoise> <!-- (Vector3): standard deviation of the additive Gaussian acceleration noise -->
+      <rateOffset>0.0 0.0 0.0</rateOffset> <!-- (Vector3): constant rate offset -->
+      <rateDrift>0.0 0.0 0.0</rateDrift> <!-- (Vector3): standard deviation of the rate drift error -->
+      <rateDriftFrequency>0.0 0.0 0.0</rateDriftFrequency> <!-- (Vector3): mean frequency of the rate drift  staviti na nulu-->
+      <rateGaussianNoise>0.0 0.0 0.0</rateGaussianNoise> <!-- (Vector3): standard deviation of the additive Gaussian rate noise -->
+      <headingOffset>0.0</headingOffset> <!-- (double): constant heading offset -->
+      <headingDrift>0.0</headingDrift> <!-- (double): standard deviation of the heading drift error -->
+      <headingDriftFrequency>0.0</headingDriftFrequency> <!-- (double): mean frequency of the heading drift  staviti na nulu-->
+      <headingGaussianNoise>0.0</headingGaussianNoise> <!-- (double): standard deviation of the heading additive Gaussian noise -->
+      <rpyOffsets>0.0 0.0 0.0</rpyOffsets> <!-- (Vector3): if non-zero, used to calculate accelOffset and headingOffset so that resulting roll, pitch and yaw errors correspond to this values when the platform is leveled (for compatibility with gazebo_plugins) -->
+    </plugin>
+  </gazebo>
   <!-- Attitude2Motion plugin -->
   <gazebo>

File: morus_description/urdf/morus.base.urdf.xacro (robot description, xacro)
@@ -202,5 +202,5 @@
   <xacro:transmisija
     trans_number="0"
-    joint_name="joint_baseToFixed_left">
+    joint_name="joint_fixedToMiddle_left">
   </xacro:transmisija>
   <xacro:transmisija
@@ -210,5 +210,5 @@
   <xacro:transmisija
     trans_number="2"
-    joint_name="joint_baseToFixed_right">
+    joint_name="joint_fixedToMiddle_right">
   </xacro:transmisija>
   <xacro:transmisija

File: morus_description/urdf/morus.urdf.xacro (robot description, xacro)
@@ -271,3 +271,20 @@
     <xacro:insert_block name="link_inertia"/>
   </xacro:manipulator>
+  <!-- Add transmission for joints -->
+  <xacro:transmisija
+    trans_number="0"
+    joint_name="joint_fixedToMiddle_left">
+  </xacro:transmisija>
+  <xacro:transmisija
+    trans_number="1"
+    joint_name="joint_middleToEnd_left">
+  </xacro:transmisija>
+  <xacro:transmisija
+    trans_number="2"
+    joint_name="joint_fixedToMiddle_right">
+  </xacro:transmisija>
+  <xacro:transmisija
+    trans_number="3"
+    joint_name="joint_middleToEnd_right">
+  </xacro:transmisija>
 </robot>

File: morus_description/urdf/multirotor_base.urdf.xacro (robot description, xacro)
@@ -1,15 +1,4 @@
 <?xml version="1.0"?>
 <robot xmlns:xacro="http://ros.org/wiki/xacro">
-  <!-- Main multirotor link -->
-  <xacro:property name="link_inertia">
-    <inertia
-    ixx="${(link_length * link_mass)/12}"
-    iyy="${(link_length * link_mass)/12}"
-    izz="${(link_length * link_mass)/12}"
-    ixy="0.0" ixz="0.0" iyz="0.0" />
-  </xacro:property>
-  <xacro:property name="PI" value="3.14" />
-  <xacro:property name="link_length" value="0.5" />
-  <xacro:property name="link_mass" value="1" />
   <xacro:macro name="multirotor_base_macro"
     params="robot_namespace mass body_width body_height mesh_file mesh_file_mass *inertia">
