Commit message: Fix joint controller

File: morus_description/urdf/morus.gazebo.xacro (robot description, xacro)
@@ -60,5 +60,5 @@
   </gazebo>
   <!-- Start publishing GM status msgs-->
-    <gazebo>
+    <!--gazebo>
     <plugin filename="libmorus_gazebo_gm_status.so" name="gm_status_1">
       <gmID> 1 </gmID>
@@ -91,5 +91,5 @@
       <motorConstant>0.000456874</motorConstant>
     </plugin>
-  </gazebo>
+  </gazebo-->
   <!-- Mount first generic pose sensor-->
   <xacro:odometry_plugin_macro

File: morus_description/urdf/morus.urdf.xacro (robot description, xacro)
@@ -28,4 +28,7 @@
   <xacro:property name="cos45" value="0.7071" />
   <xacro:property name="PI" value="3.14" />
+  <!-- Include properties -->
+  <xacro:property name="enable_rotors" value="false" />
+  <xacro:property name="enable_mass" value="false" />
   <!-- Property Blocks -->
   <xacro:property name="body_inertia">
@@ -79,149 +82,153 @@
     <xacro:insert_block name="body_inertia" />
   </xacro:multirotor_base_macro>
-  <!-- Instantiate rotors -->
-  <xacro:vertical_rotor
-    robot_namespace="$(arg name)"
-    suffix="front"
-    direction="cw"
-    motor_constant="${motor_constant}"
-    moment_constant="${moment_constant}"
-    parent="base_link"
-    mass_rotor="${mass_rotor}"
-    radius_rotor="${radius_rotor}"
-    time_constant="${time_constant}"
-    max_rot_velocity="${max_rot_velocity}"
-    motor_number="0"
-    rotor_drag_coefficient="${rotor_drag_coefficient}"
-    rolling_moment_coefficient="${rolling_moment_coefficient}"
-    color="Red">
-    <origin xyz="${arm_length+arm_offset} 0 ${propeler_offset}" rpy="0 0 0" />
-    <xacro:insert_block name="rotor_inertia" />
-  </xacro:vertical_rotor>
-  <xacro:vertical_rotor
-    robot_namespace="$(arg name)"
-    suffix="left"
-    direction="ccw"
-    motor_constant="${motor_constant}"
-    moment_constant="${moment_constant}"
-    parent="base_link"
-    mass_rotor="${mass_rotor}"
-    radius_rotor="${radius_rotor}"
-    time_constant="${time_constant}"
-    max_rot_velocity="${max_rot_velocity}"
-    motor_number="1"
-    rotor_drag_coefficient="${rotor_drag_coefficient}"
-    rolling_moment_coefficient="${rolling_moment_coefficient}"
-    color="Blue">
-    <origin xyz="0 ${arm_length+arm_offset} ${propeler_offset}" rpy="0 0 0" />
-    <xacro:insert_block name="rotor_inertia" />
-  </xacro:vertical_rotor>
-  <xacro:vertical_rotor
-    robot_namespace="$(arg name)"
-    suffix="back"
-    direction="cw"
-    motor_constant="${motor_constant}"
-    moment_constant="${moment_constant}"
-    parent="base_link"
-    mass_rotor="${mass_rotor}"
-    radius_rotor="${radius_rotor}"
-    time_constant="${time_constant}"
-    max_rot_velocity="${max_rot_velocity}"
-    motor_number="2"
-    rotor_drag_coefficient="${rotor_drag_coefficient}"
-    rolling_moment_coefficient="${rolling_moment_coefficient}"
-    color="Blue">
-    <origin xyz="${-(arm_length+arm_offset)} 0 ${propeler_offset}" rpy="0 0 0" />
-    <xacro:insert_block name="rotor_inertia" />
-  </xacro:vertical_rotor>
-  <xacro:vertical_rotor
-    robot_namespace="$(arg name)"
-    suffix="right"
-    direction="ccw"
-    motor_constant="${motor_constant}"
-    moment_constant="${moment_constant}"
-    parent="base_link"
-    mass_rotor="${mass_rotor}"
-    radius_rotor="${radius_rotor}"
-    time_constant="${time_constant}"
-    max_rot_velocity="${max_rot_velocity}"
-    motor_number="3"
-    rotor_drag_coefficient="${rotor_drag_coefficient}"
-    rolling_moment_coefficient="${rolling_moment_coefficient}"
-    color="Blue">
-    <origin xyz="0 ${-(arm_length+arm_offset)} ${propeler_offset}" rpy="0 0 0" />
-    <xacro:insert_block name="rotor_inertia" />
-  </xacro:vertical_rotor>
-  <!-- Instantiate movable mass 0-->
-  <!--xacro:movable_mass
-    mass_number="0"
-    parent="base_link"
-    mass="${movable_mass_mass}"
-    dimension="${movable_mass_dimension}"
-    color="Red"
-    x_axis="1"
-    y_axis="0"
-    z_axis="0"
-    orientation="${PI}">
-    <origin xyz="${(arm_length/2+arm_offset)} 0.0 ${movable_mass_offset}" rpy="0 0 0" />
-    <xacro:insert_block name="movable_mass_inertia"/>
-  </xacro:movable_mass-->
-  <!-- Instantiate movable mass 1 -->
-  <!--xacro:movable_mass
-    mass_number="1"
-    parent="base_link"
-    mass="${movable_mass_mass}"
-    dimension="${movable_mass_dimension}"
-    color="Blue"
-    x_axis="0"
-    y_axis="1"
-    z_axis="0"
-    orientation="${PI/2}">
-    <origin xyz="0.0 ${(arm_length/2+arm_offset)} ${movable_mass_offset}" rpy="0 0 0" />
-    <xacro:insert_block name="movable_mass_inertia"/>
-  </xacro:movable_mass-->
-  <!-- Instantiate movable mass 2-->
-  <!--xacro:movable_mass
-    mass_number="2"
-    parent="base_link"
-    mass="${movable_mass_mass}"
-    dimension="${movable_mass_dimension}"
-    color="Blue"
-    x_axis="-1"
-    y_axis="0"
-    z_axis="0"
-    orientation="${PI}">>
-    <origin xyz="${-(arm_length/2+arm_offset)} 0.0 ${movable_mass_offset}" rpy="0 0 0" />
-    <xacro:insert_block name="movable_mass_inertia"/>
-  </xacro:movable_mass-->
-  <!-- Instantiate movable mass 3 -->
-  <!--xacro:movable_mass
-    mass_number="3"
-    parent="base_link"
-    mass="${movable_mass_mass}"
-    dimension="${movable_mass_dimension}"
-    color="Blue"
-    x_axis="0"
-    y_axis="-1"
-    z_axis="0"
-    orientation="${PI/2}">>
-    <origin xyz="0.0 ${-(arm_length/2+arm_offset)} ${movable_mass_offset}" rpy="0 0 0" />
-    <xacro:insert_block name="movable_mass_inertia"/>
-  </xacro:movable_mass-->
-  <!--xacro:transmisija
-    trans_number="0"
-    joint_name="stick_to_movable_mass_0">
-  </xacro:transmisija>
-  <xacro:transmisija
-    trans_number="1"
-    joint_name="stick_to_movable_mass_1">
-  </xacro:transmisija>
-  <xacro:transmisija
-    trans_number="2"
-    joint_name="stick_to_movable_mass_2">
-  </xacro:transmisija>
-  <xacro:transmisija
-    trans_number="3"
-    joint_name="stick_to_movable_mass_3">
-  </xacro:transmisija-->
+  <group if="${enable_rotors}">
+    <!-- Instantiate rotors -->
+    <xacro:vertical_rotor
+      robot_namespace="$(arg name)"
+      suffix="front"
+      direction="cw"
+      motor_constant="${motor_constant}"
+      moment_constant="${moment_constant}"
+      parent="base_link"
+      mass_rotor="${mass_rotor}"
+      radius_rotor="${radius_rotor}"
+      time_constant="${time_constant}"
+      max_rot_velocity="${max_rot_velocity}"
+      motor_number="0"
+      rotor_drag_coefficient="${rotor_drag_coefficient}"
+      rolling_moment_coefficient="${rolling_moment_coefficient}"
+      color="Red">
+      <origin xyz="${arm_length+arm_offset} 0 ${propeler_offset}" rpy="0 0 0" />
+      <xacro:insert_block name="rotor_inertia" />
+    </xacro:vertical_rotor>
+    <xacro:vertical_rotor
+      robot_namespace="$(arg name)"
+      suffix="left"
+      direction="ccw"
+      motor_constant="${motor_constant}"
+      moment_constant="${moment_constant}"
+      parent="base_link"
+      mass_rotor="${mass_rotor}"
+      radius_rotor="${radius_rotor}"
+      time_constant="${time_constant}"
+      max_rot_velocity="${max_rot_velocity}"
+      motor_number="1"
+      rotor_drag_coefficient="${rotor_drag_coefficient}"
+      rolling_moment_coefficient="${rolling_moment_coefficient}"
+      color="Blue">
+      <origin xyz="0 ${arm_length+arm_offset} ${propeler_offset}" rpy="0 0 0" />
+      <xacro:insert_block name="rotor_inertia" />
+    </xacro:vertical_rotor>
+    <xacro:vertical_rotor
+      robot_namespace="$(arg name)"
+      suffix="back"
+      direction="cw"
+      motor_constant="${motor_constant}"
+      moment_constant="${moment_constant}"
+      parent="base_link"
+      mass_rotor="${mass_rotor}"
+      radius_rotor="${radius_rotor}"
+      time_constant="${time_constant}"
+      max_rot_velocity="${max_rot_velocity}"
+      motor_number="2"
+      rotor_drag_coefficient="${rotor_drag_coefficient}"
+      rolling_moment_coefficient="${rolling_moment_coefficient}"
+      color="Blue">
+      <origin xyz="${-(arm_length+arm_offset)} 0 ${propeler_offset}" rpy="0 0 0" />
+      <xacro:insert_block name="rotor_inertia" />
+    </xacro:vertical_rotor>
+    <xacro:vertical_rotor
+      robot_namespace="$(arg name)"
+      suffix="right"
+      direction="ccw"
+      motor_constant="${motor_constant}"
+      moment_constant="${moment_constant}"
+      parent="base_link"
+      mass_rotor="${mass_rotor}"
+      radius_rotor="${radius_rotor}"
+      time_constant="${time_constant}"
+      max_rot_velocity="${max_rot_velocity}"
+      motor_number="3"
+      rotor_drag_coefficient="${rotor_drag_coefficient}"
+      rolling_moment_coefficient="${rolling_moment_coefficient}"
+      color="Blue">
+      <origin xyz="0 ${-(arm_length+arm_offset)} ${propeler_offset}" rpy="0 0 0" />
+      <xacro:insert_block name="rotor_inertia" />
+    </xacro:vertical_rotor>
+  </group>
+  <group if="${enable_mass}">
+    <!-- Instantiate movable mass 0-->
+    <xacro:movable_mass
+      mass_number="0"
+      parent="base_link"
+      mass="${movable_mass_mass}"
+      dimension="${movable_mass_dimension}"
+      color="Red"
+      x_axis="1"
+      y_axis="0"
+      z_axis="0"
+      orientation="${PI}">
+      <origin xyz="${(arm_length/2+arm_offset)} 0.0 ${movable_mass_offset}" rpy="0 0 0" />
+      <xacro:insert_block name="movable_mass_inertia"/>
+    </xacro:movable_mass>
+    <!-- Instantiate movable mass 1 -->
+    <xacro:movable_mass
+      mass_number="1"
+      parent="base_link"
+      mass="${movable_mass_mass}"
+      dimension="${movable_mass_dimension}"
+      color="Blue"
+      x_axis="0"
+      y_axis="1"
+      z_axis="0"
+      orientation="${PI/2}">
+      <origin xyz="0.0 ${(arm_length/2+arm_offset)} ${movable_mass_offset}" rpy="0 0 0" />
+      <xacro:insert_block name="movable_mass_inertia"/>
+    </xacro:movable_mass>
+    <!-- Instantiate movable mass 2-->
+    <xacro:movable_mass
+      mass_number="2"
+      parent="base_link"
+      mass="${movable_mass_mass}"
+      dimension="${movable_mass_dimension}"
+      color="Blue"
+      x_axis="-1"
+      y_axis="0"
+      z_axis="0"
+      orientation="${PI}">>
+      <origin xyz="${-(arm_length/2+arm_offset)} 0.0 ${movable_mass_offset}" rpy="0 0 0" />
+      <xacro:insert_block name="movable_mass_inertia"/>
+    </xacro:movable_mass>
+    <!-- Instantiate movable mass 3 -->
+    <xacro:movable_mass
+      mass_number="3"
+      parent="base_link"
+      mass="${movable_mass_mass}"
+      dimension="${movable_mass_dimension}"
+      color="Blue"
+      x_axis="0"
+      y_axis="-1"
+      z_axis="0"
+      orientation="${PI/2}">>
+      <origin xyz="0.0 ${-(arm_length/2+arm_offset)} ${movable_mass_offset}" rpy="0 0 0" />
+      <xacro:insert_block name="movable_mass_inertia"/>
+    </xacro:movable_mass>
+    <xacro:transmisija
+      trans_number="0"
+      joint_name="stick_to_movable_mass_0">
+    </xacro:transmisija>
+    <xacro:transmisija
+      trans_number="1"
+      joint_name="stick_to_movable_mass_1">
+    </xacro:transmisija>
+    <xacro:transmisija
+      trans_number="2"
+      joint_name="stick_to_movable_mass_2">
+    </xacro:transmisija>
+    <xacro:transmisija
+      trans_number="3"
+      joint_name="stick_to_movable_mass_3">
+    </xacro:transmisija>
+  </group>
   <xacro:property name="land_gear_inertia">
     <inertia

File: morus_description/urdf/multirotor_base.urdf.xacro (robot description, xacro)
@@ -360,5 +360,5 @@
       <child link="link_middle_${suffix}" />
       <origin xyz="0 0 ${-(link_length/4 + link_width/2)}" rpy="0 0 0"/>
-      <limit upper="1.79769e+308" lower="-1.79769e+308" effort="-1" velocity="-1"/>
+      <limit upper="1.79769e+308" lower="-1.79769e+308" effort="20" velocity="2"/>
       <axis xyz="0 0 1" />
     </joint>
@@ -371,5 +371,5 @@
       <child link="link_end_${suffix}" />
       <origin xyz="0 ${-link_length + link_width/2} 0" rpy="0 0 0"/>
-      <limit upper="1.79769e+308" lower="-1.79769e+308" effort="-1" velocity="-1" />
+      <limit upper="1.79769e+308" lower="-1.79769e+308" effort="20" velocity="2" />
       <axis xyz="0 0 1" />
     </joint>

Commit message: Add rotors, flying(?)

File: morus_description/urdf/morus.gazebo.xacro (robot description, xacro)
@@ -60,5 +60,5 @@
   </gazebo>
   <!-- Start publishing GM status msgs-->
-    <!--gazebo>
+  <gazebo>
     <plugin filename="libmorus_gazebo_gm_status.so" name="gm_status_1">
       <gmID> 1 </gmID>
@@ -91,5 +91,5 @@
       <motorConstant>0.000456874</motorConstant>
     </plugin>
-  </gazebo-->
+  </gazebo>
   <!-- Mount first generic pose sensor-->
   <xacro:odometry_plugin_macro

File: morus_description/urdf/morus.urdf.xacro (robot description, xacro)
@@ -11,5 +11,5 @@
   <xacro:property name="arm_length" value="0.515" /> <!-- [m] -->
   <xacro:property name="arm_offset" value="0.1" /> <!-- [m] -->
-  <xacro:property name="propeler_offset" value="0.325" /> <!-- [m] -->
+  <xacro:property name="propeler_offset" value="0.5" /> <!--0.325 [m] -->
   <xacro:property name="rotor_offset_top" value="0.037" /> <!-- [m] -->
   <xacro:property name="radius_rotor" value="0.33" /> <!-- [m] -->
@@ -70,12 +70,12 @@
   <!-- Payload properties-->
   <xacro:property name="payload_mass" value="2" />
-  <xacro:property name="payload_length" value="0.1" />
-  <xacro:property name="payload_radius" value="0.05" />
+  <xacro:property name="payload_length" value="0.2" />
+  <xacro:property name="payload_radius" value="0.08" />
   <!-- Payload modelled as a solid cylinder -->
   <xacro:property name="payload_inertia">
     <inertia
-    ixx="${( (3 * payload_radius * payload_radius + payload_length * payload_length) * link_mass) / 12}"
-    iyy="${( (3 * payload_radius * payload_radius + payload_length * payload_length) * link_mass) / 12}"
-    izz="${ (payload_radius * payload_radius * link_mass) / 2}"
+    ixx="${( (3 * payload_radius * payload_radius + payload_length * payload_length) * link_mass/2 ) / 12}"
+    iyy="${( (3 * payload_radius * payload_radius + payload_length * payload_length) * link_mass/2 ) / 12}"
+    izz="${ (payload_radius * payload_radius * link_mass/2 ) / 2}"
     ixy="0.0" ixz="0.0" iyz="0.0" />
   </xacro:property>
@@ -86,5 +86,5 @@
   <xacro:property name="q2_right" value="2.0596"/>
   <!-- Include features -->
-  <xacro:property name="enable_rotors" value="false" />
+  <xacro:property name="enable_rotors" value="true" />
   <xacro:property name="enable_mass" value="false" />
   <!-- Included URDF Files -->
@@ -100,5 +100,4 @@
     <xacro:insert_block name="body_inertia" />
   </xacro:multirotor_base_macro>
-  <group if="${enable_rotors}">
     <!-- Instantiate rotors -->
     <xacro:vertical_rotor
@@ -117,5 +116,5 @@
       rolling_moment_coefficient="${rolling_moment_coefficient}"
       color="Red">
-      <origin xyz="${arm_length+arm_offset} 0 ${propeler_offset}" rpy="0 0 0" />
+      <origin xyz="${arm_length+arm_offset + 0.1} 0 ${propeler_offset}" rpy="0 0 0" />
       <xacro:insert_block name="rotor_inertia" />
     </xacro:vertical_rotor>
@@ -135,5 +134,5 @@
       rolling_moment_coefficient="${rolling_moment_coefficient}"
       color="Blue">
-      <origin xyz="0 ${arm_length+arm_offset} ${propeler_offset}" rpy="0 0 0" />
+      <origin xyz="0 ${arm_length+arm_offset + 0.1} ${propeler_offset}" rpy="0 0 0" />
       <xacro:insert_block name="rotor_inertia" />
     </xacro:vertical_rotor>
@@ -152,6 +151,6 @@
       rotor_drag_coefficient="${rotor_drag_coefficient}"
       rolling_moment_coefficient="${rolling_moment_coefficient}"
-      color="Blue">
-      <origin xyz="${-(arm_length+arm_offset)} 0 ${propeler_offset}" rpy="0 0 0" />
+      color="Red">
+      <origin xyz="${-(arm_length+arm_offset + 0.1)} 0 ${propeler_offset}" rpy="0 0 0" />
       <xacro:insert_block name="rotor_inertia" />
     </xacro:vertical_rotor>
@@ -171,8 +170,7 @@
       rolling_moment_coefficient="${rolling_moment_coefficient}"
       color="Blue">
-      <origin xyz="0 ${-(arm_length+arm_offset)} ${propeler_offset}" rpy="0 0 0" />
+      <origin xyz="0 ${-(arm_length+arm_offset + 0.1)} ${propeler_offset}" rpy="0 0 0" />
       <xacro:insert_block name="rotor_inertia" />
     </xacro:vertical_rotor>
-  </group>
   <group if="${enable_mass}">
     <!-- Instantiate movable mass 0-->
@@ -317,7 +315,17 @@
     parent="link_end_left"
     link_length="${link_length}"
-    payload_mass="${payload_mass}"
+    payload_mass="${payload_mass/2}"
     payload_length="${payload_length}"
-    payload_radius="${payload_radius}">
+    payload_radius="${payload_radius}"
+    suffix="left">
+    <xacro:insert_block name="payload_inertia"/>
+  </xacro:payload>
+  <xacro:payload
+    parent="link_end_right"
+    link_length="${link_length}"
+    payload_mass="${payload_mass/2}"
+    payload_length="${payload_length}"
+    payload_radius="${payload_radius}"
+    suffix="right">
     <xacro:insert_block name="payload_inertia"/>
   </xacro:payload>

File: morus_description/urdf/multirotor_base.urdf.xacro (robot description, xacro)
@@ -99,5 +99,5 @@
       <axis xyz="0 0 1" />
       <!-- TODO(ff): not currently set because it's not yet supported -->
-      <!-- <limit effort="2000" velocity="${max_rot_velocity}" /> -->
+      <limit effort="2000" velocity="${max_rot_velocity}"/>
       <parent link="${parent}" />
       <child link="rotor_${motor_number}" />
@@ -108,18 +108,20 @@
     <link name="rotor_${motor_number}">
       <inertial>
+        <origin xyz="0 0 0" rpy="0 0 0" />
         <mass value="${mass_rotor}" /> <!-- [kg] -->
         <xacro:insert_block name="inertia" />
       </inertial>
       <visual>
-        <!-- origin xyz="10 10 10" rpy="0 0 0" /-->
+        <origin xyz="0 0 0" rpy="0 0 0" />
         <xacro:insert_block name="origin" />
         <geometry>
-          <cylinder length="0.005" radius="${radius_rotor}"/> <!-- [m] -->
-          <!--mesh filename="package://morus_description/meshes/propeller_${direction}.dae"
-            scale="0.0025 0.0025 0.0025" /-->
+          <!--cylinder length="0.005" radius="${radius_rotor}"/--> <!-- [m] -->
+          <mesh filename="package://morus_description/meshes/propeller_${direction}.dae"
+            scale="0.0025 0.0025 0.0025" />
           <!--box size="${2*radius_rotor} 4 0.005"/-->
         </geometry>
       </visual>
       <collision>
+        <origin xyz="0 0 0" rpy="0 0 0" />
         <geometry>
           <cylinder length="0.005" radius="${radius_rotor}" /> <!-- [m] -->
@@ -303,10 +305,10 @@
       <inertial>
         <mass value="${link_mass}" />
-        <origin rpy="0 0 0" xyz="${link_length/2 - link_width/2} 0 0"/>
+        <origin rpy="0 0 0" xyz="${link_length/2} 0 0"/>
         <!--origin rpy="0 0 0" xyz="0 0 0"/-->
         <xacro:insert_block name="inertia"/>
       </inertial>
       <visual>
-        <origin rpy="0 0 0" xyz="${link_length/2 - link_width/2} 0 0"/>
+        <origin rpy="0 0 0" xyz="${link_length/2} 0 0"/>
         <geometry>
            <box size="${link_length} ${link_width} ${link_width}"/>
@@ -314,5 +316,5 @@
      </visual>
       <collision name='collision'>
-        <origin rpy="0 0 0" xyz="${link_length/2 - link_width/2} 0 0"/>
+        <origin rpy="0 0 0" xyz="${link_length/2} 0 0"/>
         <geometry>
            <box size="${link_length} ${link_width} ${link_width}"/>
@@ -339,10 +341,10 @@
         </geometry>
       </visual>
-      <!--collision name='collision'>
+      <collision name='collision'>
         <origin xyz="${link_length/2} 0 0" rpy="0 0 0"/>
         <geometry>
            <box size="${link_length} ${link_width} ${link_width}"/>
         </geometry>
-      </collision-->
+      </collision>
     </link>
     <gazebo reference="link_end_${suffix}">
@@ -376,5 +378,5 @@
       <parent link="link_middle_${suffix}" />
       <child link="link_end_${suffix}" />
-      <origin xyz="${link_length - link_width/2} 0 0" rpy="0 0 0"/>
+      <origin xyz="${link_length} 0 0" rpy="0 0 0"/>
       <limit upper="1.79769e+308" lower="-1.79769e+308" effort="10" velocity="1" />
       <axis xyz="0 0 1" />
@@ -391,6 +393,6 @@
   -->
   <xacro:macro name="payload"
-    params="parent link_length payload_mass payload_length payload_radius *inertia">
-    <link name="payload">
+    params="parent link_length payload_mass payload_length payload_radius suffix *inertia">
+    <link name="payload_${suffix}">
      <inertial>
         <mass value="${payload_mass}" />
@@ -414,7 +416,7 @@
       </collision>
     </link>
-    <joint name="joint_endToPayload" type="fixed">
+    <joint name="joint_endToPayload_${suffix}" type="fixed">
         <parent link="${parent}"/>
-        <child link="payload"/>
+        <child link="payload_${suffix}"/>
         <origin rpy="0 0 0" xyz="${link_length} 0 0"/>
     </joint>
