Commit message: Add initial position flag

File: morus_description/urdf/morus.urdf.xacro (robot description, xacro)
@@ -28,7 +28,4 @@
   <xacro:property name="cos45" value="0.7071" />
   <xacro:property name="PI" value="3.14" />
-  <!-- Include properties -->
-  <xacro:property name="enable_rotors" value="false" />
-  <xacro:property name="enable_mass" value="false" />
   <!-- Property Blocks -->
   <xacro:property name="body_inertia">
@@ -61,13 +58,34 @@
   <!-- Manipulator properties-->
   <xacro:property name="link_length" value="0.5" />
-  <xacro:property name="link_mass" value="1" />
+  <xacro:property name="link_mass" value="0.1"/>
   <xacro:property name="link_width" value="0.05" />
+  <!-- Slender rod along y - axis, rotating about its end -->
   <xacro:property name="link_inertia">
     <inertia
-    ixx="${(link_length * link_mass)/12}"
-    iyy="${(link_length * link_mass)/12}"
-    izz="${(link_length * link_mass)/12}"
+    ixx="${(link_length * link_length * link_mass)/3}"
+    iyy="0"
+    izz="${(link_length * link_length * link_mass)/3}"
     ixy="0.0" ixz="0.0" iyz="0.0" />
   </xacro:property>
+  <!-- Payload properties-->
+  <xacro:property name="payload_mass" value="2" />
+  <xacro:property name="payload_length" value="0.1" />
+  <xacro:property name="payload_radius" value="0.05" />
+  <!-- Payload modelled as a solid cylinder -->
+  <xacro:property name="payload_inertia">
+    <inertia
+    ixx="${( (3 * payload_radius * payload_radius + payload_length * payload_length) * link_mass) / 12}"
+    iyy="${( (3 * payload_radius * payload_radius + payload_length * payload_length) * link_mass) / 12}"
+    izz="${ (payload_radius * payload_radius * link_mass) / 2}"
+    ixy="0.0" ixz="0.0" iyz="0.0" />
+  </xacro:property>
+  <!--define initial conditions -->
+  <xacro:property name="q1_left" value="1.0298"/>
+  <xacro:property name="q2_left" value="-2.0596"/>
+  <xacro:property name="q1_right" value="-1.0298"/>
+  <xacro:property name="q2_right" value="2.0596"/>
+  <!-- Include features -->
+  <xacro:property name="enable_rotors" value="false" />
+  <xacro:property name="enable_mass" value="false" />
   <!-- Included URDF Files -->
   <xacro:include filename="$(find morus_description)/urdf/multirotor_base.urdf.xacro" />
@@ -265,5 +283,5 @@
     parent="base_link"
     suffix="left">
-    <origin xyz="${-(arm_length)} 0 ${-(link_length/2)}" rpy="0 0 0" />
+    <origin xyz="${-(arm_length)} 0 ${-(link_length/2)}" rpy="0 0 0"/>
     <xacro:insert_block name="link_inertia"/>
   </xacro:manipulator>
@@ -275,5 +293,5 @@
     parent="base_link"
     suffix="right">
-    <origin xyz="${arm_length} 0 ${-(link_length/2)}" rpy="0 0 0" />
+    <origin xyz="${arm_length} 0 ${-(link_length/2)}" rpy="0 0 ${PI}"/>
     <xacro:insert_block name="link_inertia"/>
   </xacro:manipulator>
@@ -295,3 +313,12 @@
     joint_name="joint_middleToEnd_right">
   </xacro:transmisija>
+  <!-- Add payload to the specified joint -->
+  <xacro:payload
+    parent="link_end_left"
+    link_length="${link_length}"
+    payload_mass="${payload_mass}"
+    payload_length="${payload_length}"
+    payload_radius="${payload_radius}">
+    <xacro:insert_block name="payload_inertia"/>
+  </xacro:payload>
 </robot>

File: morus_description/urdf/multirotor_base.urdf.xacro (robot description, xacro)
@@ -264,5 +264,5 @@
   @parent Parent link of the first (fixed) link.
   @origin Origin block determining position of the first link (its center)..
-  @intertia Intertial block definining inertia for each link.
+  @intertia Inertial block definining inertia for each link.
   -->
   <xacro:macro name="manipulator"
@@ -273,7 +273,11 @@
     <link name='link_fixed_${suffix}'>
       <inertial>
-        <mass value="1" />
-        <xacro:insert_block name="inertia"/>
+        <mass value="${link_mass/2}" />
         <origin xyz="0 0 0" rpy="0 0 0"/>
+        <inertia
+          ixx="${(link_length/2 * link_length/2 * link_mass/2)/12}"
+          iyy="${(link_length/2 * link_mass/2)/12}"
+          izz="${(link_length/2 * link_mass/2)/12}"
+          ixy="0.0" ixz="0.0" iyz="0.0" />
       </inertial>
       <visual>
@@ -298,16 +302,17 @@
     <link name='link_middle_${suffix}'>
       <inertial>
-        <mass value="1" />
+        <mass value="${link_mass}" />
+        <origin rpy="0 0 0" xyz="${link_length/2 - link_width/2} 0 0"/>
+        <!--origin rpy="0 0 0" xyz="0 0 0"/-->
         <xacro:insert_block name="inertia"/>
-        <origin rpy="0 0 0" xyz="0 ${-link_length/2 + link_width/2} 0"/>
-      </inertial>
-      <visual>
-        <origin rpy="0 0 0" xyz="0 ${-link_length/2 + link_width/2} 0"/>
-        <geometry>
-           <box size="${link_width} ${link_length} ${link_width}"/>
+      </inertial>
+      <visual>
+        <origin rpy="0 0 0" xyz="${link_length/2 - link_width/2} 0 0"/>
+        <geometry>
+           <box size="${link_length} ${link_width} ${link_width}"/>
         </geometry>
      </visual>
       <collision name='collision'>
-        <origin rpy="0 0 0" xyz="0 ${-link_length/2 + link_width/2} 0"/>
+        <origin rpy="0 0 0" xyz="${link_length/2 - link_width/2} 0 0"/>
         <geometry>
            <box size="${link_length} ${link_width} ${link_width}"/>
@@ -323,20 +328,21 @@
     <link name='link_end_${suffix}'>
       <inertial>
-        <mass value="1"/>
+        <mass value="${link_mass}"/>
         <xacro:insert_block name="inertia"/>
-        <origin xyz="0 ${-link_length/2} 0" rpy="0 0 0"/>
-      </inertial>
-      <visual>
-        <origin xyz="0 ${-link_length/2} 0" rpy="0 0 0"/>
-        <geometry>
-           <box size="${link_width} ${link_length} ${link_width}"/>
-        </geometry>
-      </visual>
-      <collision name='collision'>
-        <origin xyz="0 ${-link_length/2} 0" rpy="0 0 0"/>
-        <geometry>
-           <box size="${link_width} ${link_length} ${link_width}"/>
-        </geometry>
-      </collision>
+        <origin xyz="${link_length/2} 0 0" rpy="0 0 0"/>
+        <!--origin xyz="0 0 0" rpy="0 0 0"/-->
+      </inertial>
+      <visual>
+        <origin xyz="${link_length/2} 0 0" rpy="0 0 0"/>
+        <geometry>
+           <box size="${link_length} ${link_width} ${link_width}"/>
+        </geometry>
+      </visual>
+      <!--collision name='collision'>
+        <origin xyz="${link_length/2} 0 0" rpy="0 0 0"/>
+        <geometry>
+           <box size="${link_length} ${link_width} ${link_width}"/>
+        </geometry>
+      </collision-->
     </link>
     <gazebo reference="link_end_${suffix}">
@@ -360,5 +366,5 @@
       <child link="link_middle_${suffix}" />
       <origin xyz="0 0 ${-(link_length/4 + link_width/2)}" rpy="0 0 0"/>
-      <limit upper="1.79769e+308" lower="-1.79769e+308" effort="20" velocity="2"/>
+      <limit upper="1.79769e+308" lower="-1.79769e+308" effort="10" velocity="1"/>
       <axis xyz="0 0 1" />
     </joint>
@@ -370,8 +376,47 @@
       <parent link="link_middle_${suffix}" />
       <child link="link_end_${suffix}" />
-      <origin xyz="0 ${-link_length + link_width/2} 0" rpy="0 0 0"/>
-      <limit upper="1.79769e+308" lower="-1.79769e+308" effort="20" velocity="2" />
+      <origin xyz="${link_length - link_width/2} 0 0" rpy="0 0 0"/>
+      <limit upper="1.79769e+308" lower="-1.79769e+308" effort="10" velocity="1" />
       <axis xyz="0 0 1" />
     </joint>
   </xacro:macro>
+  <!-- Spawns a mass at the end of one specified manipulator.
+    Payload block is modelled as a cylinder.
+  @parent Reference to parent link - the link on which the payload is connected.
+  @link_length Length of the parent link.
+  @payload_mass Mass of the payload
+  @payload_length Length of the payload
+  @payload_radius Radius of the payload
+  @inertia Inertia of the payload.
+  -->
+  <xacro:macro name="payload"
+    params="parent link_length payload_mass payload_length payload_radius *inertia">
+    <link name="payload">
+     <inertial>
+        <mass value="${payload_mass}" />
+        <!--origin rpy="0 0 0" xyz="0 ${-payload_length/2 + link_width/2} 0"/-->
+        <origin rpy="0 0 0" xyz="0 0 0"/>
+        <xacro:insert_block name="inertia"/>
+      </inertial>
+      <visual>
+        <!--origin rpy="0 0 0" xyz="0 ${-link_length/2 + link_width/2} 0"/-->
+        <origin rpy="0 0 0" xyz="0 0 0"/>
+        <geometry>
+           <cylinder length="${payload_length}" radius="${payload_radius}"/>
+        </geometry>
+     </visual>
+      <collision name='collision'>
+        <origin rpy="0 0 0" xyz="0 0 0"/>
+        <!--origin rpy="0 0 0" xyz="0 ${-link_length/2 + link_width/2} 0"/-->
+        <geometry>
+           <cylinder length="${payload_length}" radius="${payload_radius}"/>
+        </geometry>
+      </collision>
+    </link>
+    <joint name="joint_endToPayload" type="fixed">
+        <parent link="${parent}"/>
+        <child link="payload"/>
+        <origin rpy="0 0 0" xyz="${link_length} 0 0"/>
+    </joint>
+  </xacro:macro>
 </robot>

Commit message: Fix manipulator positioning

File: morus_description/urdf/morus.urdf.xacro (robot description, xacro)
@@ -79,4 +79,11 @@
     izz="${ (payload_radius * payload_radius * link_mass/2 ) / 2}"
     ixy="0.0" ixz="0.0" iyz="0.0" />
+  </xacro:property>
+  <xacro:property name="payload_inertia_1">
+     <inertia
+     ixx="${(payload_mass/2 * payload_length * payload_length)/6}"
+     iyy="${(payload_mass/2 * payload_length * payload_length)/6}"
+     izz="${(payload_mass/2 * payload_length * payload_length)/6}"
+     ixy="0.0" ixz="0.0"  iyz="0.0" /> <!-- [kg*m^2] [kg*m^2] [kg*m^2] [kg*m^2] [kg*m^2] [kg*m^2] -->
   </xacro:property>
   <!--define initial conditions -->

Commit message: Add: Reference filter, 0Div Fix, new UAV mesh, circle demo

File: morus_description/urdf/morus.urdf.xacro (robot description, xacro)
@@ -3,5 +3,5 @@
   <!-- Properties -->
   <xacro:property name="rotor_velocity_slowdown_sim" value="10" />
-  <xacro:property name="mesh_file" value="MORUS_UAV_without_mass.dae" />
+  <xacro:property name="mesh_file" value="MORUS_without_legs.dae" />
   <xacro:property name="mesh_file_mass" value="MORUS_mass.dae" />
   <xacro:property name="mass" value="30" />  <!-- [kg] -->
@@ -11,5 +11,5 @@
   <xacro:property name="arm_length" value="0.515" /> <!-- [m] -->
   <xacro:property name="arm_offset" value="0.1" /> <!-- [m] -->
-  <xacro:property name="propeler_offset" value="0.5" /> <!--0.325 [m] -->
+  <xacro:property name="propeler_offset" value="0.3" /> <!--0.325 [m] -->
   <xacro:property name="rotor_offset_top" value="0.037" /> <!-- [m] -->
   <xacro:property name="radius_rotor" value="0.33" /> <!-- [m] -->
@@ -123,5 +123,5 @@
       rolling_moment_coefficient="${rolling_moment_coefficient}"
       color="Red">
-      <origin xyz="${arm_length+arm_offset + 0.1} 0 ${propeler_offset}" rpy="0 0 0" />
+      <origin xyz="${arm_length+arm_offset} 0 ${propeler_offset}" rpy="0 0 0" />
       <xacro:insert_block name="rotor_inertia" />
     </xacro:vertical_rotor>
@@ -141,5 +141,5 @@
       rolling_moment_coefficient="${rolling_moment_coefficient}"
       color="Blue">
-      <origin xyz="0 ${arm_length+arm_offset + 0.1} ${propeler_offset}" rpy="0 0 0" />
+      <origin xyz="0 ${arm_length+arm_offset} ${propeler_offset}" rpy="0 0 0" />
       <xacro:insert_block name="rotor_inertia" />
     </xacro:vertical_rotor>
@@ -159,5 +159,5 @@
       rolling_moment_coefficient="${rolling_moment_coefficient}"
       color="Red">
-      <origin xyz="${-(arm_length+arm_offset + 0.1)} 0 ${propeler_offset}" rpy="0 0 0" />
+      <origin xyz="${-(arm_length+arm_offset)} 0 ${propeler_offset}" rpy="0 0 0" />
       <xacro:insert_block name="rotor_inertia" />
     </xacro:vertical_rotor>
@@ -177,5 +177,5 @@
       rolling_moment_coefficient="${rolling_moment_coefficient}"
       color="Blue">
-      <origin xyz="0 ${-(arm_length+arm_offset + 0.1)} ${propeler_offset}" rpy="0 0 0" />
+      <origin xyz="0 ${-(arm_length+arm_offset)} ${propeler_offset}" rpy="0 0 0" />
       <xacro:insert_block name="rotor_inertia" />
     </xacro:vertical_rotor>

File: morus_description/urdf/multirotor_base.urdf.xacro (robot description, xacro)
@@ -16,8 +16,9 @@
       </inertial>
       <visual>
-        <origin xyz="0 0 0.125" rpy="0 0 0" />
-        <geometry>
-          <!-- mesh filename="package://morus_description/meshes/${mesh_file}" scale="1 1 1" / -->
-          <box size="${body_width} ${body_width} ${body_height}" /> <!-- [m] [m] [m] -->
+        <!-- Origin of the modified mesh, comment if using box -->
+        <origin xyz="0 0 0.1" rpy="0 0 0" />
+        <geometry>
+          <mesh filename="package://morus_description/meshes/${mesh_file}" scale="1 1 1" />
+          <!--box size="${body_width} ${body_width} ${body_height}" /--> <!-- [m] [m] [m] -->
         </geometry>
       </visual>
