Commit message: Camera added

File: morus_description/urdf/morus.urdf.xacro (robot description, xacro)
@@ -72,4 +72,14 @@
   <xacro:property name="payload_length" value="0.2" />
   <xacro:property name="payload_radius" value="0.08" />
+  <!-- Camera properties -->
+  <xacro:property name="camera_link" value="0.05" />
+  <xacro:property name="camera_inertia">
+    <inertia
+    ixx="1e-6"
+    iyy="1e-6"
+    izz="1e-6"
+    ixy="0.0" ixz="0.0" iyz="0.0" />
+  </xacro:property>
+  <xacro:property name="camera_mass" value="1e-5"/>
   <!-- Payload modelled as a solid cylinder -->
   <xacro:property name="payload_inertia">
@@ -337,3 +347,10 @@
     <xacro:insert_block name="payload_inertia"/>
   </xacro:payload>
+  <xacro:cam
+    camera_link="${camera_link}"
+    camera_mass="${camera_mass}"
+    parent="base_link">
+    <origin xyz="0 0 -1" rpy="0 ${-PI/2} 0"/>
+    <xacro:insert_block name="camera_inertia"/>
+  </xacro:cam>
 </robot>

File: morus_description/urdf/multirotor_base.urdf.xacro (robot description, xacro)
@@ -191,42 +191,211 @@
     </link>
   </xacro:macro>
-   <!-- camera -->
-  <xacro:macro name="camera_macro" params="robot_namespace">
-    <!-- joint -->
+  <!--Spawns manipulator:
+  Manipulator is modeled as a 2DOF manipulator where first link is
+  fixed to the base. Other two links are conecteted with
+  revolute joints.
+  @link_length Length of link.
+  @link_width Width of link.
+  @link_mass Link mass.
+  @parent Parent link of the first (fixed) link.
+  @origin Origin block determining position of the first link (its center)..
+  @intertia Inertial block definining inertia for each link.
+  -->
+  <xacro:macro name="manipulator"
+  params="link_length link_width link_mass parent suffix *origin *inertia">
+    <!--_____________________________________________________________-->
+    <!--LINK1-->
+    <!--_____________________________________________________________-->
+    <link name='link_fixed_${suffix}'>
+      <inertial>
+        <mass value="${link_mass/2}" />
+        <origin xyz="0 0 0" rpy="0 0 0"/>
+        <inertia
+          ixx="${(link_length/2 * link_length/2 * link_mass/2)/12}"
+          iyy="${(link_length/2 * link_mass/2)/12}"
+          izz="${(link_length/2 * link_mass/2)/12}"
+          ixy="0.0" ixz="0.0" iyz="0.0" />
+      </inertial>
+      <visual>
+        <origin xyz="0 0 0" rpy="0 0 0"/>
+        <geometry>
+           <box size="${link_width} ${link_width} ${link_length/2}"/>
+        </geometry>
+      </visual>
+      <collision name='collision'>
+        <origin xyz="0 0 0" rpy="0 0 0"/>
+        <geometry>
+           <box size="${link_width} ${link_width} ${link_length/2}"/>
+        </geometry>
+      </collision>
+    </link>
+    <gazebo reference="link_fixed_${suffix}">
+      <material>Gazebo/Red</material>
+    </gazebo>
+    <!--_____________________________________________________________-->
+    <!--LINK2-->
+    <!--_____________________________________________________________-->
+    <link name='link_middle_${suffix}'>
+      <inertial>
+        <mass value="${link_mass}" />
+        <origin rpy="0 0 0" xyz="${link_length/2} 0 0"/>
+        <!--origin rpy="0 0 0" xyz="0 0 0"/-->
+        <xacro:insert_block name="inertia"/>
+      </inertial>
+      <visual>
+        <origin rpy="0 0 0" xyz="${link_length/2} 0 0"/>
+        <geometry>
+           <box size="${link_length} ${link_width} ${link_width}"/>
+        </geometry>
+     </visual>
+      <collision name='collision'>
+        <origin rpy="0 0 0" xyz="${link_length/2} 0 0"/>
+        <geometry>
+           <box size="${link_length} ${link_width} ${link_width}"/>
+        </geometry>
+      </collision>
+    </link>
+    <gazebo reference="link_middle_${suffix}">
+      <material>Gazebo/Blue</material>
+    </gazebo>
+    <!--_____________________________________________________________-->
+    <!--LINK3-->
+    <!--_____________________________________________________________-->
+    <link name='link_end_${suffix}'>
+      <inertial>
+        <mass value="${link_mass}"/>
+        <xacro:insert_block name="inertia"/>
+        <origin xyz="${link_length/2} 0 0" rpy="0 0 0"/>
+        <!--origin xyz="0 0 0" rpy="0 0 0"/-->
+      </inertial>
+      <visual>
+        <origin xyz="${link_length/2} 0 0" rpy="0 0 0"/>
+        <geometry>
+           <box size="${link_length} ${link_width} ${link_width}"/>
+        </geometry>
+      </visual>
+      <collision name='collision'>
+        <origin xyz="${link_length/2} 0 0" rpy="0 0 0"/>
+        <geometry>
+           <box size="${link_length} ${link_width} ${link_width}"/>
+        </geometry>
+      </collision>
+    </link>
+    <gazebo reference="link_end_${suffix}">
+      <material>Gazebo/Green</material>
+    </gazebo>
+    <!--_____________________________________________________________-->
+    <!--JOINT_baseToFixed-->
+    <!--Fixed joint connecting base to first link (fixed)-->
+    <!--_____________________________________________________________-->
+    <joint name="joint_baseToFixed_${suffix}" type="fixed">
+        <xacro:insert_block name="origin"/>
+        <parent link="${parent}"/>
+        <child link="link_fixed_${suffix}"/>
+    </joint>
+    <!--_____________________________________________________________-->
+    <!--JOINT_fixedtoMiddle-->
+    <!--Revolute joint connecting fixed link to middle link-->
+    <!--_____________________________________________________________-->
+    <joint name='joint_fixedToMiddle_${suffix}' type='revolute'>
+      <parent link="link_fixed_${suffix}" />
+      <child link="link_middle_${suffix}" />
+      <origin xyz="0 0 ${-(link_length/4 + link_width/2)}" rpy="0 0 0"/>
+      <limit upper="1.79769e+308" lower="-1.79769e+308" effort="10" velocity="1"/>
+      <axis xyz="0 0 1" />
+    </joint>
+    <!--_____________________________________________________________-->
+    <!--JOINT_middleToEnd-->
+    <!--Revolute joint connecting middle link to end link.-->
+    <!--_____________________________________________________________-->
+    <joint name="joint_middleToEnd_${suffix}" type="revolute">
+      <parent link="link_middle_${suffix}" />
+      <child link="link_end_${suffix}" />
+      <origin xyz="${link_length} 0 0" rpy="0 0 0"/>
+      <limit upper="1.79769e+308" lower="-1.79769e+308" effort="10" velocity="1" />
+      <axis xyz="0 0 1" />
+    </joint>
+  </xacro:macro>
+  <!-- Spawns a mass at the end of one specified manipulator.
+    Payload block is modelled as a cylinder.
+  @parent Reference to parent link - the link on which the payload is connected.
+  @link_length Length of the parent link.
+  @payload_mass Mass of the payload
+  @payload_length Length of the payload
+  @payload_radius Radius of the payload
+  @inertia Inertia of the payload.
+  -->
+  <xacro:macro name="payload"
+    params="parent link_length payload_mass payload_length payload_radius suffix *inertia">
+    <link name="payload_${suffix}">
+     <inertial>
+        <mass value="${payload_mass}" />
+        <origin rpy="0 0 0" xyz="0 0 0"/>
+        <xacro:insert_block name="inertia"/>
+      </inertial>
+      <visual>
+        <origin rpy="0 0 0" xyz="0 0 0"/>
+        <geometry>
+           <cylinder length="${payload_length}" radius="${payload_radius}"/>
+        </geometry>
+     </visual>
+      <collision name='collision'>
+        <origin rpy="0 0 0" xyz="0 0 0"/>
+        <geometry>
+           <cylinder length="${payload_length}" radius="${payload_radius}"/>
+        </geometry>
+      </collision>
+    </link>
+    <joint name="joint_endToPayload_${suffix}" type="fixed">
+        <parent link="${parent}"/>
+        <child link="payload_${suffix}"/>
+        <origin rpy="0 0 0" xyz="${link_length} 0 0"/>
+    </joint>
+  </xacro:macro>
+  <!-- Camera macro. Adds a box representing a camera below the UAV
+  @param camera_link Length of the camera box
+  @param camera_mass Mass of the camera
+  @param parent Parent link on which the camera will be fixed
+  @param *origin Block argument defining the origin of the camera with
+  reference to the parent link.
+  @param *inertia Block argument defining camera inertia.
+  -->
+  <xacro:macro name="cam" params="camera_link camera_mass parent *origin *inertia">
+    <!-- Camera link -->
+    <link name="camera_box">
+      <!--collision>
+        <origin xyz="0 0 0" rpy="0 0 0"/>
+        <geometry>
+          <box size="${camera_link} ${camera_link} ${camera_link}"/>
+        </geometry>
+      </collision-->
+      <visual>
+        <origin xyz="0 0 0" rpy="0 0 0"/>
+        <geometry>
+          <box size="${camera_link} ${camera_link} ${camera_link}"/>
+        </geometry>
+        <material name="red"/>
+      </visual>
+      <inertial>
+        <mass value="${camera_mass}" />
+        <origin xyz="0 0 0" rpy="0 0 0"/>
+        <xacro:insert_block name="inertia"/>
+      </inertial>
+    </link>
+    <!-- Camera joint with reference to the parent link -->
     <joint name="camera_joint" type="fixed">
-      <axis xyz="0 1 0" />
-      <origin xyz="0 0 0.2" rpy="0 0 0" />
-      <parent link="base_link" />
-      <child link="camera_link" />
-    </joint>
-    <!-- link -->
-    <link name="camera_link">
-      <collision>
-        <origin xyz="0 0 0" rpy="0 0 0" />
-        <geometry>
-          <box size="0.1 0.1 0.1" />
-        </geometry>
-      </collision>
-      <visual>
-        <origin xyz="0 0 0" rpy="0 0 0" />
-        <geometry>
-          <box size="0.1 0.1 0.1" />
-        </geometry>
-        <material name="red" />
-      </visual>
-      <inertial>
-        <mass value="1e-5" />
-        <origin xyz="0 0 0" rpy="0 0 0" />
-        <inertia ixx="1e-6" ixy="0" ixz="0" iyy="1e-6" iyz="0" izz="1e-6" />
-      </inertial>
-    </link>
-    <gazebo reference="camera_link">
+      <xacro:insert_block name="origin"/>
+      <parent link="${parent}"/>
+      <child link="camera_box"/>
+    </joint>
+    <!-- camera -->
+    <gazebo reference="camera_box">
       <sensor type="camera" name="camera1">
         <update_rate>30.0</update_rate>
         <camera name="head">
-          <horizontal_fov>2</horizontal_fov>
+          <horizontal_fov>1.3962634</horizontal_fov>
           <image>
             <width>800</width>
-            <height>600</height>
+            <height>800</height>
             <format>R8G8B8</format>
           </image>
@@ -244,8 +413,8 @@
           <alwaysOn>true</alwaysOn>
           <updateRate>0.0</updateRate>
-          <cameraName>${robot_namespace}/camera1</cameraName>
+          <cameraName>morus/camera1</cameraName>
           <imageTopicName>image_raw</imageTopicName>
           <cameraInfoTopicName>camera_info</cameraInfoTopicName>
-          <frameName>camera_link</frameName>
+          <frameName>camera_box</frameName>
           <hackBaseline>0.07</hackBaseline>
           <distortionK1>0.0</distortionK1>
@@ -258,168 +427,3 @@
     </gazebo>
   </xacro:macro>
-  <!--Spawns manipulator:
-  Manipulator is modeled as a 2DOF manipulator where first link is
-  fixed to the base. Other two links are conecteted with
-  revolute joints.
-  @link_length Length of link.
-  @link_width Width of link.
-  @link_mass Link mass.
-  @parent Parent link of the first (fixed) link.
-  @origin Origin block determining position of the first link (its center)..
-  @intertia Inertial block definining inertia for each link.
-  -->
-  <xacro:macro name="manipulator"
-  params="link_length link_width link_mass parent suffix *origin *inertia">
-    <!--_____________________________________________________________-->
-    <!--LINK1-->
-    <!--_____________________________________________________________-->
-    <link name='link_fixed_${suffix}'>
-      <inertial>
-        <mass value="${link_mass/2}" />
-        <origin xyz="0 0 0" rpy="0 0 0"/>
-        <inertia
-          ixx="${(link_length/2 * link_length/2 * link_mass/2)/12}"
-          iyy="${(link_length/2 * link_mass/2)/12}"
-          izz="${(link_length/2 * link_mass/2)/12}"
-          ixy="0.0" ixz="0.0" iyz="0.0" />
-      </inertial>
-      <visual>
-        <origin xyz="0 0 0" rpy="0 0 0"/>
-        <geometry>
-           <box size="${link_width} ${link_width} ${link_length/2}"/>
-        </geometry>
-      </visual>
-      <collision name='collision'>
-        <origin xyz="0 0 0" rpy="0 0 0"/>
-        <geometry>
-           <box size="${link_width} ${link_width} ${link_length/2}"/>
-        </geometry>
-      </collision>
-    </link>
-    <gazebo reference="link_fixed_${suffix}">
-      <material>Gazebo/Red</material>
-    </gazebo>
-    <!--_____________________________________________________________-->
-    <!--LINK2-->
-    <!--_____________________________________________________________-->
-    <link name='link_middle_${suffix}'>
-      <inertial>
-        <mass value="${link_mass}" />
-        <origin rpy="0 0 0" xyz="${link_length/2} 0 0"/>
-        <!--origin rpy="0 0 0" xyz="0 0 0"/-->
-        <xacro:insert_block name="inertia"/>
-      </inertial>
-      <visual>
-        <origin rpy="0 0 0" xyz="${link_length/2} 0 0"/>
-        <geometry>
-           <box size="${link_length} ${link_width} ${link_width}"/>
-        </geometry>
-     </visual>
-      <collision name='collision'>
-        <origin rpy="0 0 0" xyz="${link_length/2} 0 0"/>
-        <geometry>
-           <box size="${link_length} ${link_width} ${link_width}"/>
-        </geometry>
-      </collision>
-    </link>
-    <gazebo reference="link_middle_${suffix}">
-      <material>Gazebo/Blue</material>
-    </gazebo>
-    <!--_____________________________________________________________-->
-    <!--LINK3-->
-    <!--_____________________________________________________________-->
-    <link name='link_end_${suffix}'>
-      <inertial>
-        <mass value="${link_mass}"/>
-        <xacro:insert_block name="inertia"/>
-        <origin xyz="${link_length/2} 0 0" rpy="0 0 0"/>
-        <!--origin xyz="0 0 0" rpy="0 0 0"/-->
-      </inertial>
-      <visual>
-        <origin xyz="${link_length/2} 0 0" rpy="0 0 0"/>
-        <geometry>
-           <box size="${link_length} ${link_width} ${link_width}"/>
-        </geometry>
-      </visual>
-      <collision name='collision'>
-        <origin xyz="${link_length/2} 0 0" rpy="0 0 0"/>
-        <geometry>
-           <box size="${link_length} ${link_width} ${link_width}"/>
-        </geometry>
-      </collision>
-    </link>
-    <gazebo reference="link_end_${suffix}">
-      <material>Gazebo/Green</material>
-    </gazebo>
-    <!--_____________________________________________________________-->
-    <!--JOINT_baseToFixed-->
-    <!--Fixed joint connecting base to first link (fixed)-->
-    <!--_____________________________________________________________-->
-    <joint name="joint_baseToFixed_${suffix}" type="fixed">
-        <xacro:insert_block name="origin"/>
-        <parent link="${parent}"/>
-        <child link="link_fixed_${suffix}"/>
-    </joint>
-    <!--_____________________________________________________________-->
-    <!--JOINT_fixedtoMiddle-->
-    <!--Revolute joint connecting fixed link to middle link-->
-    <!--_____________________________________________________________-->
-    <joint name='joint_fixedToMiddle_${suffix}' type='revolute'>
-      <parent link="link_fixed_${suffix}" />
-      <child link="link_middle_${suffix}" />
-      <origin xyz="0 0 ${-(link_length/4 + link_width/2)}" rpy="0 0 0"/>
-      <limit upper="1.79769e+308" lower="-1.79769e+308" effort="10" velocity="1"/>
-      <axis xyz="0 0 1" />
-    </joint>
-    <!--_____________________________________________________________-->
-    <!--JOINT_middleToEnd-->
-    <!--Revolute joint connecting middle link to end link.-->
-    <!--_____________________________________________________________-->
-    <joint name="joint_middleToEnd_${suffix}" type="revolute">
-      <parent link="link_middle_${suffix}" />
-      <child link="link_end_${suffix}" />
-      <origin xyz="${link_length} 0 0" rpy="0 0 0"/>
-      <limit upper="1.79769e+308" lower="-1.79769e+308" effort="10" velocity="1" />
-      <axis xyz="0 0 1" />
-    </joint>
-  </xacro:macro>
-  <!-- Spawns a mass at the end of one specified manipulator.
-    Payload block is modelled as a cylinder.
-  @parent Reference to parent link - the link on which the payload is connected.
-  @link_length Length of the parent link.
-  @payload_mass Mass of the payload
-  @payload_length Length of the payload
-  @payload_radius Radius of the payload
-  @inertia Inertia of the payload.
-  -->
-  <xacro:macro name="payload"
-    params="parent link_length payload_mass payload_length payload_radius suffix *inertia">
-    <link name="payload_${suffix}">
-     <inertial>
-        <mass value="${payload_mass}" />
-        <!--origin rpy="0 0 0" xyz="0 ${-payload_length/2 + link_width/2} 0"/-->
-        <origin rpy="0 0 0" xyz="0 0 0"/>
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